File: hardware/2S3P Power Board TI BQ25798/2S3P Power Board TI BQ25798.kicad_pcb (KiCad board)
At the start: 4 copper layers, 8.9 x 4.3 mm, 108 parts, among them J201 B02B-XASK-1 (LF)(SN), J202 B02B-XASK-1 (LF)(SN), J301 USB, J501 B02B-XASK-1 (LF)(SN), J701 504050-1291, J702 504050-0491, Q401 CSD17581Q3A, Q402 CSD17581Q3A, Q403 CSD17581Q3A, Q404 CSD17581Q3A, U201 BQ25798RQMR, U501 1042, U502 1042, U503 1042, U504 1042, U505 1042, U506 1042, U601 TLV76733DRVx, U602 TLV76750DRVx

Commit message: Checkpointing work after feedback from team
Parts:
- removed C201, C202, C203, C205, C206, C214, C216, C217, C218, C219, C220, C221: 10u, Capacitor_SMD:C_0603_1608Metric
- removed C204, C207, C209, C210, C213: 0.1u, Capacitor_SMD:C_0402_1005Metric
- removed C208: 4.7u, Capacitor_SMD:C_0805_2012Metric
- removed C211, C212: 0.047u, Capacitor_SMD:C_0402_1005Metric
- removed C215, C401, C402: 1n, Capacitor_SMD:C_0402_1005Metric
- removed C601, C602: 1u, Capacitor_SMD:C_0805_2012Metric
- removed C603, C604: 2.2u, Capacitor_SMD:C_0805_2012Metric
- removed D201: Green LED, LED_SMD:LED_0603_1608Metric
- removed D401, D402: 12V, Diode_SMD:D_SOD-523
- removed D601, D602: Orange LED, LED_SMD:LED_1210_3225Metric
- removed J201, J202, J501: B02B-XASK-1 (LF)(SN), footprints:B02BXASK1LFSN
- removed J301: USB, footprints:CONN_124018612112A_AMP
- removed J701: 504050-1291, footprints:5040501291
- removed J702: 504050-0491, footprints:5040500491
- removed JP201: 3P Header, footprints:HDRV3W64P0X254_1X3_762X254X869P
- removed L201: 1uH, Inductor_SMD:L_12x12mm_H8mm
- removed Q401, Q402, Q403, Q404: CSD17581Q3A, footprints:Q3A_TEX
- removed R201: 2.21k, Resistor_SMD:R_0402_1005Metric
- removed R202: 5.24k, Resistor_SMD:R_0402_1005Metric
- removed R203: 30.31k, Resistor_SMD:R_0603_1608Metric
- removed R204, R205, R207, R212, R213: 0.01, Resistor_SMD:R_2512_6332Metric
- removed R206, R208, R210: 10k, Resistor_SMD:R_0402_1005Metric
- removed R209: 6.2k, Resistor_SMD:R_0603_1608Metric
- removed R211: 100, Resistor_SMD:R_0603_1608Metric
- removed R401, R402: 294, Resistor_SMD:R_0603_1608Metric
- removed R601: 68, Resistor_SMD:R_0402_1005Metric
- removed R602: 150, Resistor_SMD:R_0402_1005Metric
- removed TH201: 10k NTC, Resistor_SMD:R_0402_1005Metric
- removed TP201, TP202, TP203, TP204, TP205, TP206, TP212, TP213, TP215, TP216, TP303, TP304, TP405, TP406, TP502, TP503, TP504: White, TestPoint:TestPoint_Keystone_5000-5004_Miniature
- removed TP207, TP208, TP301, TP306, TP403, TP404: Black, TestPoint:TestPoint_Keystone_5000-5004_Miniature
- removed TP209, TP210, TP211, TP214, TP305, TP505, TP601, TP602: Ring, TestPoint:TestPoint_Keystone_5019_Minature
- removed TP302, TP401, TP402, TP501, TP603, TP604: Red, TestPoint:TestPoint_Keystone_5000-5004_Miniature
- removed U201: BQ25798RQMR, footprints:RQM0029A-MFG
- removed U501, U502, U503, U504, U505, U506: 1042, footprints:KEYSTONE-1042
- removed U601: TLV76733DRVx, Package_SON:WSON-6-1EP_2x2mm_P0.65mm_EP1x1.6mm_ThermalVias
- removed U602: TLV76750DRVx, Package_SON:WSON-6-1EP_2x2mm_P0.65mm_EP1x1.6mm_ThermalVias
Other:
- board outline removed
