File: hardware/power/power_board/batteries_2s3p.kicad_sch (KiCad schematic)
At the start: 12 parts, among them J501 B02B-XASK-1 (LF)(SN), U501 1042, U502 1042, U503 1042, U504 1042, U505 1042, U506 1042

Commit message: Changed interconnect from battery to power board to use the 10-pin Pico-Lock receptacle and cable.
Parts:
- removed J501: B02B-XASK-1 (LF)(SN), footprints:B02BXASK1LFSN, symbol JST B02B-XASK-1 (LF)(SN):B02B-XASK-1__LF__SN_
- removed TP501: Red, TestPoint:TestPoint_Keystone_5000-5004_Miniature, symbol Connector:TestPoint
- removed TP502, TP503, TP504: White, TestPoint:TestPoint_Keystone_5000-5004_Miniature, symbol Connector:TestPoint
- removed TP505: Ring, TestPoint:TestPoint_Keystone_5019_Minature, symbol Connector:TestPoint
- removed U501, U502, U503, U504, U505, U506: 1042, footprints:KEYSTONE-1042, symbol Keystone 1042:1042
