File: electrical/pcb_design/power_board/usb.kicad_sch (KiCad schematic)
At the start: 7 parts, among them J301 Molex_430450612

Commit message: Updated test point symbols in 2s3p battery board and power board
Parts:
- TP301, TP306: footprint TestPoint:TestPoint_Keystone_5000-5004_Miniature -> footprints:Keystone_5001; symbol Connector:TestPoint -> TVSC:TestPoint_Keystone_5001; Color (none) -> Black
- TP302: footprint TestPoint:TestPoint_Keystone_5000-5004_Miniature -> footprints:Keystone_5000; symbol Connector:TestPoint -> TVSC:TestPoint_Keystone_5000; Color (none) -> Red
- TP303, TP304: footprint TestPoint:TestPoint_Keystone_5000-5004_Miniature -> footprints:Keystone_5002; symbol Connector:TestPoint -> TVSC:TestPoint_Keystone_5002; Color (none) -> White
- TP305: footprint TestPoint:TestPoint_Keystone_5019_Minature -> footprints:Keystone_5019; symbol Connector:TestPoint -> TVSC:TestPoint_Keystone_5019; Color (none) -> Ring
Changed lines of the file:
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@@
     )
   )
-  (symbol (lib_id "Connector:TestPoint") (at 137.16 87.63 0) (unit 1)
+  (symbol (lib_id "TVSC:TestPoint_Keystone_5001") (at 137.16 87.63 0) (unit 1)
     (in_bom yes) (on_board yes) (dnp no) (fields_autoplaced)
     (property "Reference" "TP306" (at 139.7 83.058 0)
@@
       (effects (font (size 1.27 1.27)) (justify left))
     )
-    (property "Footprint" "TestPoint:TestPoint_Keystone_5000-5004_Miniature" (at 142.24 87.63 0)
-      (effects (font (size 1.27 1.27)) hide)
-    )
-    (property "Datasheet" "~" (at 142.24 87.63 0)
+    (property "Footprint" "footprints:Keystone_5001" (at 142.24 87.63 0)
+      (effects (font (size 1.27 1.27)) hide)
+    )
+    (property "Datasheet" "https://www.keyelco.com/product.cfm/product_id/1310" (at 142.24 87.63 0)
+      (effects (font (size 1.27 1.27)) hide)
+    )
+    (property "MPN" "C238122" (at 137.16 87.63 0)
+      (effects (font (size 1.27 1.27)) hide)
+    )
+    (property "Manufacturer" "Keystone" (at 137.16 87.63 0)
+      (effects (font (size 1.27 1.27)) hide)
+    )
+    (property "Purpose" "" (at 137.16 87.63 0)
+      (effects (font (size 1.27 1.27)) hide)
+    )
+    (property "Color" "Black" (at 142.24 87.63 0)
+      (effects (font (size 1.27 1.27)) hide)
+    )
+    (property "Manufacturer Part Number" "5001" (at 137.16 87.63 0)
       (effects (font (size 1.27 1.27)) hide)
     )
@@
       (effects (font (size 1.27 1.27)) hide)
     )
-    (property "MPN" "C238122" (at 137.16 87.63 0)
-      (effects (font (size 1.27 1.27)) hide)
-    )
-    (property "Manufacturer" "Keystone" (at 137.16 87.63 0)
-      (effects (font (size 1.27 1.27)) hide)
-    )
-    (property "Manufacturer Part Number" "5001" (at 137.16 87.63 0)
-      (effects (font (size 1.27 1.27)) hide)
-    )
-    (property "Purpose" "" (at 137.16 87.63 0)
-      (effects (font (size 1.27 1.27)) hide)
-    )
     (pin "1")
     (instances
@@
     )
   )
-  (symbol (lib_id "Connector:TestPoint") (at 137.16 95.25 180) (unit 1)
+  (symbol (lib_id "TVSC:TestPoint_Keystone_5001") (at 137.16 95.25 180) (unit 1)
     (in_bom yes) (on_board yes) (dnp no) (fields_autoplaced)
     (property "Reference" "TP301" (at 139.7 97.282 0)
@@
       (effects (font (size 1.27 1.27)) (justify right))
     )
-    (property "Footprint" "TestPoint:TestPoint_Keystone_5000-5004_Miniature" (at 132.08 95.25 0)
-      (effects (font (size 1.27 1.27)) hide)
-    )
-    (property "Datasheet" "~" (at 132.08 95.25 0)
+    (property "Footprint" "footprints:Keystone_5001" (at 132.08 95.25 0)
+      (effects (font (size 1.27 1.27)) hide)
+    )
+    (property "Datasheet" "https://www.keyelco.com/product.cfm/product_id/1310" (at 132.08 95.25 0)
+      (effects (font (size 1.27 1.27)) hide)
+    )
+    (property "MPN" "C238122" (at 137.16 95.25 0)
+      (effects (font (size 1.27 1.27)) hide)
+    )
+    (property "Manufacturer" "Keystone" (at 137.16 95.25 0)
+      (effects (font (size 1.27 1.27)) hide)
+    )
+    (property "Purpose" "" (at 137.16 95.25 0)
+      (effects (font (size 1.27 1.27)) hide)
+    )
+    (property "Color" "Black" (at 132.08 95.25 0)
+      (effects (font (size 1.27 1.27)) hide)
+    )
+    (property "Manufacturer Part Number" "5001" (at 137.16 95.25 0)
       (effects (font (size 1.27 1.27)) hide)
     )
@@
       (effects (font (size 1.27 1.27)) hide)
     )
-    (property "MPN" "C238122" (at 137.16 95.25 0)
-      (effects (font (size 1.27 1.27)) hide)
-    )
-    (property "Manufacturer" "Keystone" (at 137.16 95.25 0)
-      (effects (font (size 1.27 1.27)) hide)
-    )
-    (property "Manufacturer Part Number" "5001" (at 137.16 95.25 0)
-      (effects (font (size 1.27 1.27)) hide)
-    )
-    (property "Purpose" "" (at 137.16 95.25 0)
-      (effects (font (size 1.27 1.27)) hide)
-    )
     (pin "1")
     (instances
@@
     )
   )
-  (symbol (lib_id "Connector:TestPoint") (at 120.65 96.52 180) (unit 1)
+  (symbol (lib_id "TVSC:TestPoint_Keystone_5002") (at 120.65 96.52 180) (unit 1)
     (in_bom yes) (on_board yes) (dnp no)
     (property "Reference" "TP304" (at 128.27 100.33 0)
@@
       (effects (font (size 1.27 1.27)) (justify left))
     )
-    (property "Footprint" "TestPoint:TestPoint_Keystone_5000-5004_Miniature" (at 115.57 96.52 0)
-      (effects (font (size 1.27 1.27)) hide)
-    )
-    (property "Datasheet" "~" (at 115.57 96.52 0)
+    (property "Footprint" "footprints:Keystone_5002" (at 115.57 96.52 0)
+      (effects (font (size 1.27 1.27)) hide)
+    )
+    (property "Datasheet" "https://www.keyelco.com/product.cfm/product_id/1311" (at 115.57 96.52 0)
       (effects (font (size 1.27 1.27)) hide)
     )
@@
       (effects (font (size 1.27 1.27)) hide)
     )
+    (property "Purpose" "" (at 120.65 96.52 0)
+      (effects (font (size 1.27 1.27)) hide)
+    )
+    (property "Color" "White" (at 115.57 96.52 0)
+      (effects (font (size 1.27 1.27)) hide)
+    )
     (property "Manufacturer Part Number" "5002" (at 120.65 96.52 0)
       (effects (font (size 1.27 1.27)) hide)
     )
     (property "Active" "Y" (at 120.65 96.52 0)
-      (effects (font (size 1.27 1.27)) hide)
-    )
-    (property "Purpose" "" (at 120.65 96.52 0)
       (effects (font (size 1.27 1.27)) hide)
     )
@@
     )
   )
-  (symbol (lib_id "Connector:TestPoint") (at 147.32 76.2 0) (unit 1)
+  (symbol (lib_id "TVSC:TestPoint_Keystone_5000") (at 147.32 76.2 0) (unit 1)
     (in_bom yes) (on_board yes) (dnp no)
     (property "Reference" "TP302" (at 148.59 71.12 0)
@@
       (effects (font (size 1.27 1.27)) (justify left))
     )
-    (property "Footprint" "TestPoint:TestPoint_Keystone_5000-5004_Miniature" (at 152.4 76.2 0)
-      (effects (font (size 1.27 1.27)) hide)
-    )
-    (property "Datasheet" "~" (at 152.4 76.2 0)
+    (property "Footprint" "footprints:Keystone_5000" (at 152.4 76.2 0)
+      (effects (font (size 1.27 1.27)) hide)
+    )
+    (property "Datasheet" "https://www.keyelco.com/product.cfm/product_id/1309" (at 152.4 76.2 0)
       (effects (font (size 1.27 1.27)) hide)
     )
@@
       (effects (font (size 1.27 1.27)) hide)
     )
+    (property "Purpose" "" (at 147.32 76.2 0)
+      (effects (font (size 1.27 1.27)) hide)
+    )
+    (property "Color" "Red" (at 152.4 76.2 0)
+      (effects (font (size 1.27 1.27)) hide)
+    )
     (property "Active" "Y" (at 147.32 76.2 0)
-      (effects (font (size 1.27 1.27)) hide)
-    )
-    (property "Purpose" "" (at 147.32 76.2 0)
       (effects (font (size 1.27 1.27)) hide)
     )
@@
     )
   )
-  (symbol (lib_id "Connector:TestPoint") (at 120.65 87.63 0) (unit 1)
+  (symbol (lib_id "TVSC:TestPoint_Keystone_5002") (at 120.65 87.63 0) (unit 1)
     (in_bom yes) (on_board yes) (dnp no) (fields_autoplaced)
     (property "Reference" "TP303" (at 123.19 83.058 0)
@@
       (effects (font (size 1.27 1.27)) (justify left))
     )
-    (property "Footprint" "TestPoint:TestPoint_Keystone_5000-5004_Miniature" (at 125.73 87.63 0)
-      (effects (font (size 1.27 1.27)) hide)
-    )
-    (property "Datasheet" "~" (at 125.73 87.63 0)
+    (property "Footprint" "footprints:Keystone_5002" (at 125.73 87.63 0)
+      (effects (font (size 1.27 1.27)) hide)
+    )
+    (property "Datasheet" "https://www.keyelco.com/product.cfm/product_id/1311" (at 125.73 87.63 0)
       (effects (font (size 1.27 1.27)) hide)
     )
@@
       (effects (font (size 1.27 1.27)) hide)
     )
+    (property "Purpose" "" (at 120.65 87.63 0)
+      (effects (font (size 1.27 1.27)) hide)
+    )
+    (property "Color" "White" (at 125.73 87.63 0)
+      (effects (font (size 1.27 1.27)) hide)
+    )
     (property "Manufacturer Part Number" "5002" (at 120.65 87.63 0)
       (effects (font (size 1.27 1.27)) hide)
@@
       (effects (font (size 1.27 1.27)) hide)
     )
-    (property "Purpose" "" (at 120.65 87.63 0)
-      (effects (font (size 1.27 1.27)) hide)
-    )
     (pin "1")
     (instances
@@
     )
   )
-  (symbol (lib_id "Connector:TestPoint") (at 154.94 101.6 90) (unit 1)
+  (symbol (lib_id "TVSC:TestPoint_Keystone_5019") (at 154.94 101.6 90) (unit 1)
     (in_bom yes) (on_board yes) (dnp no)
     (property "Reference" "TP305" (at 148.59 104.14 90)
@@
       (effects (font (size 1.27 1.27)))
     )
-    (property "Footprint" "TestPoint:TestPoint_Keystone_5019_Minature" (at 154.94 96.52 0)
-      (effects (font (size 1.27 1.27)) hide)
-    )
-    (property "Datasheet" "~" (at 154.94 96.52 0)
+    (property "Footprint" "footprints:Keystone_5019" (at 154.94 96.52 0)
+      (effects (font (size 1.27 1.27)) hide)
+    )
+    (property "Datasheet" "https://www.keyelco.com/product.cfm/product_id/1357" (at 154.94 96.52 0)
       (effects (font (size 1.27 1.27)) hide)
     )
@@
       (effects (font (size 1.27 1.27)) hide)
     )
+    (property "Purpose" "" (at 154.94 101.6 0)
+      (effects (font (size 1.27 1.27)) hide)
+    )
+    (property "Color" "Ring" (at 154.94 96.52 0)
+      (effects (font (size 1.27 1.27)) hide)
+    )
     (property "Manufacturer Part Number" "5019" (at 154.94 101.6 0)
       (effects (font (size 1.27 1.27)) hide)
@@
       (effects (font (size 1.27 1.27)) hide)
     )
-    (property "Purpose" "" (at 154.94 101.6 0)
-      (effects (font (size 1.27 1.27)) hide)
-    )
