File: electrical/pcb_design/1s3p_battery_board/1s3p_battery_board.kicad_pcb (KiCad board)
At the start: 4 copper layers, 82.5 x 82.5 mm, 92 parts, among them J1 STLINK, J2 Molex_504050-1291, J3 Molex_504050-1291, J4 Power Interconnect, Q1 CSD16342Q5A, Q2 CSD16342Q5A, Q3 CSD16342Q5A, U1 STM32L452RCTx, U2 TCAN330DR, U3 PAC1934T-I/JQ, U8 TPS63900

Commit message: Checkpoint work on 1s3p battery board.
Parts:
- removed J3: Molex_504050-1291, footprints:Bus Connector (Control)
- removed R35, R36, R40, R41: 0, Resistor_SMD:R_2512_6332Metric
- removed TP4: BOARD_LOAD_+, footprints:TestPoint_Pad_D1.5mm
- removed TP6: +3V3, footprints:TestPoint_Pad_D1.5mm
- removed TP8: VBATT, footprints:TestPoint_Pad_D1.5mm
- added C18: 10u, footprints:Nondescript_C_0603_1608Metric, F.Cu at (-37.0, 79.5)
- added C19: 10u, footprints:Nondescript_C_0603_1608Metric, F.Cu at (-37.0, 82.0)
- added C22: 100n, footprints:Nondescript_C_0402_1005Metric, F.Cu at (-25.5, 79.2)
- added C23: 100n, footprints:Nondescript_C_0402_1005Metric, F.Cu at (-25.5, 81.2)
- added C24: 10u, footprints:Nondescript_C_0603_1608Metric, F.Cu at (-37.0, 84.5)
- added C25: 10u, footprints:Nondescript_C_0603_1608Metric, F.Cu at (-37.0, 87.0)
- added C26: 100n, footprints:Nondescript_C_0402_1005Metric, F.Cu at (-25.5, 83.2)
- added C28: 100n, footprints:Nondescript_C_0402_1005Metric, F.Cu at (-25.5, 85.1)
- added C29: 10u, footprints:Nondescript_C_0603_1608Metric, F.Cu at (-37.0, 89.5)
- added C30: 10u, footprints:Nondescript_C_0603_1608Metric, F.Cu at (-33.0, 79.5)
- added C31: 10u, footprints:Nondescript_C_0603_1608Metric, F.Cu at (-33.0, 82.0)
- added C32: 0.047u, footprints:Nondescript_C_0402_1005Metric, F.Cu at (-25.5, 87.1)
- added C33: 0.047u, footprints:Nondescript_C_0402_1005Metric, F.Cu at (-25.5, 89.1)
- added C34: 100n, footprints:Nondescript_C_0402_1005Metric, F.Cu at (-25.5, 91.0)
- added C35: 10u, footprints:Nondescript_C_0603_1608Metric, F.Cu at (-33.0, 84.5)
- added C36: 10u, footprints:Nondescript_C_0603_1608Metric, F.Cu at (-33.0, 87.0)
- added C37: 10u, footprints:Nondescript_C_0603_1608Metric, F.Cu at (-33.0, 89.5)
- added C38: 10u, footprints:Nondescript_C_0603_1608Metric, F.Cu at (-29.0, 79.5)
- added C39: 10u, footprints:Nondescript_C_0603_1608Metric, F.Cu at (-29.0, 82.0)
- added C40: 10u, footprints:Nondescript_C_0603_1608Metric, F.Cu at (-29.0, 84.5)
- added C41: 10u, footprints:Nondescript_C_0603_1608Metric, F.Cu at (-29.0, 87.0)
- added C42: 100n, footprints:Nondescript_C_0402_1005Metric, F.Cu at (-25.5, 93.0)
- added D2: Blue LED, LED_SMD:LED_0603_1608Metric, F.Cu at (-30.6, 96.4)
- added J5: QTH-030-07-L-D-A, footprints:SAMTEC_QTH-030-07-L-D-A, F.Cu at (119.2, 127.0)
- added J6: QSH-030-01-L-D-A, footprints:SAMTEC_QSH-030-01-L-D-A, B.Cu at (119.2, 127.0)
- added JP7: SolderJumper_2_Open, Jumper:SolderJumper-2_P1.3mm_Open_RoundedPad1.0x1.5mm, F.Cu at (-21.9, 93.7)
- added L2: 2.2µH, Inductor_SMD:L_1008_2520Metric, F.Cu at (-21.6, 90.0)
- added Q4: CSD17581Q3A, Package_SON:VSON-8_3.3x3.3mm_P0.65mm_NexFET, B.Cu at (168.4, 42.2)
- added Q5: CSD17581Q3A, Package_SON:VSON-8_3.3x3.3mm_P0.65mm_NexFET, B.Cu at (156.7, 52.2)
- added U4: BQ25798, Package_DFN_QFN:Texas_RQM0029A_VQFN-29_4x4mm_P0.4mm, F.Cu at (-35.6, 93.8)
- added U5: TPS3840DL18DBVR, footprints:DBV0005A_L, F.Cu at (-9.36, 101.7)
- J2: value Molex_504050-1291 -> B2B-PH-K-S__LF__SN_; footprint footprints:Bus Connector (Target) -> footprints:B2BPHKSLFSN
- J4: value Power Interconnect -> USB_C_Receptacle
- PCB1: footprint footprints:Battery_Board_Shape_Space_Invader_2 -> footprints:Core_Board
- Q1, Q2, Q3: value CSD16342Q5A -> CSD17581Q3A
- R10: value 10m -> 100m; footprint Resistor_SMD:R_2512_6332Metric -> Resistor_SMD:R_0805_2012Metric
- R23, R30: value 9k31 -> R
- R24: value 10m -> 33; footprint Resistor_SMD:R_2512_6332Metric -> footprints:Nondescript_R_0402_1005Metric
- R26: value 9k31 -> 100; footprint footprints:Nondescript_R_0402_1005Metric -> Resistor_SMD:R_0402_1005Metric_Pad0.72x0.64mm_HandSolder
- R27: value 10m -> 294; footprint Resistor_SMD:R_2512_6332Metric -> Resistor_SMD:R_0402_1005Metric_Pad0.72x0.64mm_HandSolder
- R28: value 9k31 -> 294; footprint footprints:Nondescript_R_0402_1005Metric -> Resistor_SMD:R_0402_1005Metric_Pad0.72x0.64mm_HandSolder
- R29: value 10m -> 9k31; footprint Resistor_SMD:R_2512_6332Metric -> footprints:Nondescript_R_0402_1005Metric
- R31, R34: value 0 -> 9k31; footprint Resistor_SMD:R_2512_6332Metric -> footprints:Nondescript_R_0402_1005Metric
- R32, R33: value 0 -> 5k1; footprint Resistor_SMD:R_2512_6332Metric -> Resistor_SMD:R_0402_1005Metric_Pad0.72x0.64mm_HandSolder
- R38: moved to F.Cu
- R51: footprint footprints:Nondescript_R_0603_1608Metric -> footprints:Nondescript_R_0402_1005Metric
- U3: footprint footprints:UQFN-16-1EP_4x4mm_P0.65mm_EP2.6x2.6mm -> Package_DFN_QFN:UQFN-16-1EP_4x4mm_P0.65mm_EP2.6x2.6mm
- U8: footprint Package_SON:WSON-10-1EP_2.5x2.5mm_P0.5mm_EP1.2x2mm -> Package_SON:WSON-10-1EP_2.5x2.5mm_P0.5mm_EP1.2x2mm_ThermalVias
- moved J4 186.4 mm to (-29.8, -2.35)
- moved J2 100.1 mm to (72.6, 126.2)
- moved Q1 96.6 mm to (151.1, 42.2)
- moved Q3 95.8 mm to (144.0, 51.9)
- moved Q2 87.8 mm to (181.9, 52.5)
- moved R29 76.6 mm to (97.4, 73.5)
- moved TH1 65.8 mm to (105.3, 74.2)
- moved R30 64.7 mm to (106.3, 71.2)
- moved R33 57.7 mm to (106.2, 124.0)
- moved C6 52.4 mm to (210.7, 99.9)
- moved R25 52.4 mm to (212.7, 99.9)
- moved U3 52.4 mm to (210.6, 96.7)
- moved C17 52.4 mm to (213.7, 98.3)
- moved R27 47.2 mm to (105.8, 66.8)
- moved R34 44.3 mm to (106.8, 144.4)
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Connections:
- BT1 pad N: Net-(BT1-PadN) -> GND
- BT1 pad P: /Batteries/B1+ -> /Batteries/VBATT
- BT2 pad N: Net-(BT2-PadN) -> GND
- BT2 pad P: /Batteries/B2+ -> /Batteries/VBATT
- BT3 pad N: Net-(BT3-PadN) -> GND
- BT3 pad P: /Batteries/B3+ -> /Batteries/VBATT
- C5 pad 1: /Batteries/BOARD_LOAD_+ -> /Voltage Regulation/BOARD_LOAD_+
- J2 pad 1: GND -> /Batteries/EXTERNAL_VIN
- J4 pad 1: GND -> (no net)
- J4 pad 2: GND -> (no net)
- J4 pad 3: GND -> (no net)
- J4 pad 4: VBATT -> (no net)
- J4 pad 5: VBATT -> (no net)
- J4 pad 6: VBATT -> (no net)
- J4 pad 7: GND -> (no net)
- J4 pad 8: GND -> (no net)
- JP10 pad 1: /Board Identification/BOARD_ID_SENSE -> Net-(JP10-A)
- JP13 pad 1: /Board Identification/BOARD_ID_SENSE -> Net-(JP10-A)
- Q1 pad 1: GND -> Net-(D3-A)
- Q1 pad 2: GND -> Net-(D3-A)
- Q1 pad 3: GND -> Net-(D3-A)
- Q1 pad 4: /Batteries/BATTERY_1_EN -> Net-(D3-K)
- Q1 pad 5: Net-(Q1-D) -> /Batteries/USB_VIN
- Q2 pad 1: GND -> Net-(D3-A)
- Q2 pad 2: GND -> Net-(D3-A)
- Q2 pad 3: GND -> Net-(D3-A)
- Q2 pad 4: /Batteries/BATTERY_2_EN -> Net-(D3-K)
- Q2 pad 5: Net-(Q2-D) -> /Batteries/BATT_VBUS
- Q3 pad 1: GND -> Net-(D4-A)
- Q3 pad 2: GND -> Net-(D4-A)
- Q3 pad 3: GND -> Net-(D4-A)
- Q3 pad 4: /Batteries/BATTERY_3_EN -> Net-(D4-K)
- Q3 pad 5: Net-(Q3-D) -> /Batteries/EXTERNAL_VIN
- R10 pad 1: /Batteries/BOARD_LOAD_+ -> /Voltage Regulation/BOARD_LOAD_+
- R23 pad 1: VBATT -> Net-(U4-TS)
- R23 pad 2: /Batteries/BATTERY_1_EN -> GND
- R24 pad 1: VBATT -> Net-(D2-K)
- R24 pad 2: /Batteries/B1+ -> Net-(U4-STAT)
- R26 pad 1: VBATT -> Net-(U4-BATP)
- R26 pad 2: /Batteries/BATTERY_2_EN -> /Batteries/VBATT
- R27 pad 1: VBATT -> Net-(D3-K)
- R27 pad 2: /Batteries/B2+ -> Net-(U4-ACDRV1)
- R28 pad 1: VBATT -> Net-(D4-K)
- R28 pad 2: /Batteries/BATTERY_3_EN -> Net-(U4-ACDRV2)
- R29 pad 1: VBATT -> Net-(U4-PROG)
- R29 pad 2: /Batteries/B3+ -> GND
- R30 pad 1: +3V3 -> /Batteries/REGN
- R30 pad 2: /Batteries/TEMPERATURE_SENSE -> Net-(U4-TS)
- R31 pad 1: Net-(BT1-PadN) -> Net-(U4-PROG)
- R31 pad 2: Net-(Q1-D) -> GND
- R32 pad 1: Net-(BT1-PadN) -> Net-(J4-CC2)
- R33 pad 1: Net-(BT2-PadN) -> Net-(J4-CC1)
- R33 pad 2: Net-(Q2-D) -> GND
- R34 pad 1: Net-(BT2-PadN) -> +3V3
- R34 pad 2: GND -> /Batteries/BATT_INT
- TH1 pad 1: /Batteries/TEMPERATURE_SENSE -> Net-(U4-TS)
- TP5 pad 1: /Board Identification/BOARD_ID_SENSE -> Net-(JP10-A)
- TP7 pad 1: /Batteries/TEMPERATURE_SENSE -> Net-(U4-TS)
- U1 pad 16: GND -> /Board Identification/BOARD_ID_VERSION
- U1 pad 21: /Batteries/TEMPERATURE_SENSE -> unconnected-(U1-PA5-Pad21)
- U1 pad 41: unconnected-(U1-PA8-Pad41) -> /Batteries/BATT_INT
- U1 pad 50: unconnected-(U1-PA15-Pad50) -> /MCU/PERIPH_INT_2
- U1 pad 56: /Batteries/BATTERY_3_EN -> unconnected-(U1-PB4-Pad56)
- U1 pad 57: /Batteries/BATTERY_2_EN -> unconnected-(U1-PB5-Pad57)
- U1 pad 61: /Batteries/BATTERY_1_EN -> unconnected-(U1-PB8-Pad61)
- U3 pad 10: /Batteries/B2+ -> unconnected-(U3-SENSE4+-Pad10)
- U3 pad 11: /Batteries/B3+ -> /Voltage Regulation/BOARD_LOAD_+
- U3 pad 12: VBATT -> +3V3
- U3 pad 13: /Batteries/BOARD_LOAD_+ -> unconnected-(U3-SENSE2+-Pad13)
- U3 pad 14: +3V3 -> unconnected-(U3-SENSE2--Pad14)
- U3 pad 4: /Batteries/I2C_SCL -> /Batteries/I2C_SDA
- U3 pad 5: /Batteries/I2C_SDA -> /Batteries/I2C_SCL
- U3 pad 7: VBATT -> unconnected-(U3-SENSE3--Pad7)
- U3 pad 8: /Batteries/B1+ -> unconnected-(U3-SENSE3+-Pad8)
- U3 pad 9: VBATT -> unconnected-(U3-SENSE4--Pad9)
- U8 pad 6: /Batteries/BOARD_LOAD_+ -> /Voltage Regulation/BOARD_LOAD_+
Routing:
- net /Batteries/BATTERY_3_EN: track 76.0 -> 0.00 mm, vias 3 -> 0
- net /Batteries/BATTERY_2_EN: track 66.1 -> 0.00 mm, vias 3 -> 0
- net /Batteries/BATTERY_1_EN: track 64.8 -> 0.00 mm, vias 4 -> 0
- net /CTRL.SWO: track 55.3 -> 0.00 mm, vias 4 -> 0
- net /NRST: track 87.7 -> 32.7 mm, vias 2 -> 0
- net /CTRL.SWCLK: track 53.8 -> 0.00 mm, vias 2 -> 0
- net /CTRL.NRST: track 53.4 -> 0.00 mm, vias 2 -> 0
- net /CTRL.SWDIO: track 53.2 -> 0.00 mm, vias 2 -> 0
- net /SWCLK: track 88.7 -> 41.3 mm, vias 2 -> 0
- net VBATT: track 44.5 -> 0.00 mm, vias 1 -> 0
- net /SWDIO: track 92.6 -> 48.9 mm, vias 3 -> 1
- net /Batteries/BOARD_LOAD_+: track 41.2 -> 0.00 mm
- net /Batteries/TEMPERATURE_SENSE: track 37.9 -> 0.00 mm, vias 3 -> 0
- net /CTRL.BOOT0: track 37.6 -> 0.00 mm, vias 2 -> 0
- net /Batteries/B1+: track 31.8 -> 0.00 mm, vias 2 -> 0
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- added copper zone on F.Cu, net /Batteries/VBATT
- added copper zone on In2.Cu, net /Batteries/VBATT
- added copper zone on B.Cu, net /Voltage Regulation/BOARD_LOAD_+
- removed copper zone on B.Cu, net /Batteries/B1+
- removed copper zone on B.Cu, net /Batteries/B2+
- removed copper zone on B.Cu, net /Batteries/B3+
- removed copper zone on B.Cu, net /Batteries/BOARD_LOAD_+
- removed copper zone on B.Cu, net Net-(BT1-PadN)
- removed copper zone on B.Cu, net Net-(BT2-PadN)
- removed copper zone on B.Cu, net Net-(BT3-PadN)
- removed copper zone on B.Cu, net Net-(Q1-D)
- removed copper zone on B.Cu, net Net-(Q2-D)
- removed copper zone on B.Cu, net Net-(Q3-D)
- removed copper zone on B.Cu, net VBATT
- removed copper zone on F.Cu, net VBUS
- removed copper zone on In2.Cu, net VBUS
Other:
- outline, holes or cut-outs redrawn
- board text added: "X"

Commit message: Checkpoint work on 1s3p board and magnetorquer board.
Parts:
- removed C22: 100n, footprints:Nondescript_C_0402_1005Metric
- added C21: 100n, footprints:Nondescript_C_0402_1005Metric, F.Cu at (62.7, 146.0)
- Q1, Q2, Q5: value CSD17581Q3A -> CSD13385F5; footprint Package_SON:VSON-8_3.3x3.3mm_P0.65mm_NexFET -> footprints:PICOSTAR3_YJK_TEX
- Q3, Q4: value CSD17581Q3A -> CSD13385F5; footprint Package_SON:VSON-8_3.3x3.3mm_P0.65mm_NexFET -> footprints:PICOSTAR3_YJK_TEX; moved to F.Cu
- R28: moved to F.Cu
- moved J4 155.0 mm to (28.9, 141.2)
- moved Q4 150.7 mm to (59.7, 146.6), turned to 0 degrees
- moved Q3 125.0 mm to (59.7, 144.2), turned to 0 degrees
- moved R28 104.7 mm to (62.9, 144.0), turned to 0 degrees
- moved C18 69.3 mm to (31.0, 93.1)
- moved C19 69.3 mm to (31.0, 95.6)
- moved C23 69.3 mm to (42.4, 94.8)
- moved C24 69.3 mm to (31.0, 98.1)
- moved C25 69.3 mm to (31.0, 100.6)
- moved C26 69.3 mm to (42.4, 96.8)
- moved C28 69.3 mm to (42.4, 98.8)
- moved C29 69.3 mm to (31.0, 103.2)
- moved C30 69.3 mm to (35.0, 93.1)
- moved C31 69.3 mm to (35.0, 95.6)
- moved C32 69.3 mm to (42.4, 100.7)
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Connections:
- C18 pad 1: Net-(C18-Pad1) -> Net-(Q5-S)
- C19 pad 1: Net-(C18-Pad1) -> Net-(Q5-S)
- Q1 pad 1: Net-(D3-A) -> Net-(D3-K)
- Q1 pad 3: Net-(D3-A) -> /Batteries/USB_VIN
- Q2 pad 1: Net-(D3-A) -> Net-(D3-K)
- Q2 pad 3: Net-(D3-A) -> /Batteries/BATT_VBUS
- Q3 pad 1: Net-(D4-A) -> Net-(D4-K)
- Q3 pad 3: Net-(D4-A) -> /Batteries/EXTERNAL_VIN
- Q4 pad 1: Net-(D4-A) -> Net-(D4-K)
- Q4 pad 3: Net-(D4-A) -> /Batteries/BATT_VBUS
- Q5 pad 1: Net-(C18-Pad1) -> Net-(Q5-G)
- Q5 pad 2: Net-(C18-Pad1) -> Net-(Q5-S)
- Q5 pad 3: Net-(C18-Pad1) -> /Batteries/VBATT
- U4 pad 22: Net-(C18-Pad1) -> Net-(Q5-S)
- U4 pad 23: Net-(C18-Pad1) -> Net-(Q5-S)

Commit message: Checkpoint progress on battery board. Preparing to break out reusable functional modules.
Parts:
- removed J4: USB_C_Receptacle, footprints:Molex_504050-0691
- removed TP7: TEMP, footprints:TestPoint_Pad_D1.5mm
- added C22: 10u, footprints:Nondescript_C_0603_1608Metric, F.Cu at (214.3, 114.4)
- added D4: Blue LED, LED_SMD:LED_0603_1608Metric, F.Cu at (214.4, 111.9)
- added JP11: SolderJumper_2_Open, Jumper:SolderJumper-2_P1.3mm_Open_RoundedPad1.0x1.5mm, F.Cu at (53.0, 62.4)
- added JP12: SolderJumper_2_Open, Jumper:SolderJumper-2_P1.3mm_Open_RoundedPad1.0x1.5mm, F.Cu at (53.0, 66.0)
- added JP16: SolderJumper_2_Open, Jumper:SolderJumper-2_P1.3mm_Open_RoundedPad1.0x1.5mm, F.Cu at (53.0, 69.5)
- added JP17: SolderJumper_2_Open, Jumper:SolderJumper-2_P1.3mm_Open_RoundedPad1.0x1.5mm, F.Cu at (53.0, 73.0)
- added JP8: SolderJumper_2_Open, Jumper:SolderJumper-2_P1.3mm_Open_RoundedPad1.0x1.5mm, F.Cu at (53.0, 55.3)
- added JP9: SolderJumper_2_Open, Jumper:SolderJumper-2_P1.3mm_Open_RoundedPad1.0x1.5mm, F.Cu at (53.0, 58.9)
- added L3: 2.2µH, Inductor_SMD:L_1008_2520Metric, F.Cu at (74.2, 103.0)
- added L4: 2.2µH, Inductor_SMD:L_1008_2520Metric, F.Cu at (67.3, 103.0)
- added L5: 2.2µH, Inductor_SMD:L_1008_2520Metric, F.Cu at (67.3, 95.2)
- added L6: 2.2µH, Inductor_SMD:L_1008_2520Metric, F.Cu at (81.2, 95.2)
- added L7: 2.2µH, Inductor_SMD:L_1008_2520Metric, F.Cu at (74.2, 95.2)
- added L8: 2.2µH, Inductor_SMD:L_1008_2520Metric, F.Cu at (81.2, 103.0)
- added R35: 36k5, footprints:Nondescript_R_0402_1005Metric, F.Cu at (56.6, 54.5)
- added R36: 100m, Resistor_SMD:R_0805_2012Metric, F.Cu at (56.6, 56.5)
- added R40: 9k31, footprints:Nondescript_R_0402_1005Metric, F.Cu at (56.6, 58.5)
- added R41: 5k1, Resistor_SMD:R_0402_1005Metric_Pad0.72x0.64mm_HandSolder, F.Cu at (56.6, 60.5)
- added R42: 9k31, footprints:Nondescript_R_0402_1005Metric, F.Cu at (73.2, 105.8)
- added R45: 9k31, footprints:Nondescript_R_0402_1005Metric, F.Cu at (66.2, 105.8)
- added R48: 9k31, footprints:Nondescript_R_0402_1005Metric, F.Cu at (66.2, 98.1)
- added R54: 9k31, footprints:Nondescript_R_0402_1005Metric, F.Cu at (80.1, 98.1)
- added R57: 9k31, footprints:Nondescript_R_0402_1005Metric, F.Cu at (73.2, 98.1)
- added R60: 9k31, footprints:Nondescript_R_0402_1005Metric, F.Cu at (80.1, 105.8)
- added TH2: 10k NTC, footprints:Nondescript_R_0603_1608Metric, F.Cu at (57.2, 62.7)
- added TH3: 10k NTC, footprints:Nondescript_R_0603_1608Metric, F.Cu at (57.2, 65.2)
- added U10: SPV1040TTR, footprints:SOIC_1040T_STM, B.Cu at (86.8, 154.8)
- added U11: SPV1040TTR, footprints:SOIC_1040T_STM, B.Cu at (93.6, 161.2)
- added U12: LM66100DCK, Package_TO_SOT_SMD:SOT-363_SC-70-6, B.Cu at (93.6, 166.0)
- added U13: LM66100DCK, Package_TO_SOT_SMD:SOT-363_SC-70-6, B.Cu at (86.8, 158.5)
- added U14: SPV1040TTR, footprints:SOIC_1040T_STM, B.Cu at (86.8, 162.1)
- added U15: LM66100DCK, Package_TO_SOT_SMD:SOT-363_SC-70-6, B.Cu at (93.6, 170.7)
- added U16: SPV1040TTR, footprints:SOIC_1040T_STM, B.Cu at (86.8, 165.8)
- added U17: LM66100DCK, Package_TO_SOT_SMD:SOT-363_SC-70-6, B.Cu at (93.6, 175.5)
- added U18: SPV1040TTR, footprints:SOIC_1040T_STM, B.Cu at (86.8, 169.4)
- added U6: LM66100DCK, Package_TO_SOT_SMD:SOT-363_SC-70-6, B.Cu at (93.6, 151.7)
- added U7: SPV1040TTR, footprints:SOIC_1040T_STM, B.Cu at (86.8, 151.2)
- added U9: LM66100DCK, Package_TO_SOT_SMD:SOT-363_SC-70-6, B.Cu at (93.6, 156.4)
- C17, C21, C26, C34: value 100n -> 10u; footprint footprints:Nondescript_C_0402_1005Metric -> footprints:Nondescript_C_0603_1608Metric
- C19: value 10u -> 1n
- C24, C30, C4, C41: value 10u -> 100n; footprint footprints:Nondescript_C_0603_1608Metric -> footprints:Nondescript_C_0402_1005Metric
- C27: value 22u -> 0.047u; footprint footprints:Nondescript_C_0603_1608Metric -> footprints:Nondescript_C_0402_1005Metric
- C28: value 100n -> 0.047u
- C32, C33: value 0.047u -> 10u; footprint footprints:Nondescript_C_0402_1005Metric -> footprints:Nondescript_C_0603_1608Metric
- C38, C40: value 10u -> 22u
- C5: value 22u -> 100n; footprint footprints:Nondescript_C_0603_1608Metric -> footprints:Nondescript_C_0402_1005Metric
- D2: value Blue LED -> Zener
- J2: value B2B-PH-K-S__LF__SN_ -> USB_C_Receptacle
- R10: value 100m -> 9k31; footprint Resistor_SMD:R_0805_2012Metric -> footprints:Nondescript_R_0402_1005Metric
- R23: value R -> 9k31
- R24: value 33 -> 57k9
- R25: value 9k31 -> 294; footprint footprints:Nondescript_R_0402_1005Metric -> Resistor_SMD:R_0402_1005Metric_Pad0.72x0.64mm_HandSolder
- R26: value 100 -> 7k2; footprint Resistor_SMD:R_0402_1005Metric_Pad0.72x0.64mm_HandSolder -> footprints:Nondescript_R_0402_1005Metric
- R28: value 294 -> 57k9; footprint Resistor_SMD:R_0402_1005Metric_Pad0.72x0.64mm_HandSolder -> footprints:Nondescript_R_0402_1005Metric
- R30: value R -> 7k2
- R31: value 9k31 -> 57k9
- R32: value 5k1 -> 7k2; footprint Resistor_SMD:R_0402_1005Metric_Pad0.72x0.64mm_HandSolder -> footprints:Nondescript_R_0402_1005Metric
- R33: value 5k1 -> 33; footprint Resistor_SMD:R_0402_1005Metric_Pad0.72x0.64mm_HandSolder -> footprints:Nondescript_R_0402_1005Metric
- R34: value 9k31 -> 100; footprint footprints:Nondescript_R_0402_1005Metric -> Resistor_SMD:R_0402_1005Metric_Pad0.72x0.64mm_HandSolder
- R51: value 36k5 -> 5k1; footprint footprints:Nondescript_R_0402_1005Metric -> Resistor_SMD:R_0402_1005Metric_Pad0.72x0.64mm_HandSolder
- TH1: footprint footprints:Nondescript_R_0402_1005Metric -> footprints:Nondescript_R_0603_1608Metric; moved to F.Cu
- TP1: value VBUS -> TEMP
- TP3: value GND -> VBUS
- U3: value PAC1934T-I/JQ -> TPS3840DL18DBVR; footprint Package_DFN_QFN:UQFN-16-1EP_4x4mm_P0.65mm_EP2.6x2.6mm -> footprints:DBV0005A_L
- U5: value TPS3840DL18DBVR -> TPS63900; footprint footprints:DBV0005A_L -> Package_SON:WSON-10-1EP_2.5x2.5mm_P0.5mm_EP1.2x2mm_ThermalVias
- U8: value TPS63900 -> PAC1934T-I/JQ; footprint Package_SON:WSON-10-1EP_2.5x2.5mm_P0.5mm_EP1.2x2mm_ThermalVias -> Package_DFN_QFN:UQFN-16-1EP_4x4mm_P0.65mm_EP2.6x2.6mm
- moved TP3 79.3 mm to (220.1, 112.3)
- moved TH1 41.6 mm to (65.0, 64.0), turned to 0 degrees
- moved TP1 17.3 mm to (180.2, 62.0)
Connections:
- C17 pad 1: +3V3 -> /Batteries/REGN
- C17 pad 2: GND -> Net-(C17-Pad2)
- C18 pad 1: Net-(Q5-S) -> Net-(C17-Pad2)
- C19 pad 1: Net-(Q5-S) -> Net-(D2-A)
- C19 pad 2: GND -> Net-(D2-K)
- C21 pad 1: /Batteries/EXTERNAL_VIN -> /Batteries/BATT_VBUS
- C23 pad 1: /Batteries/USB_VIN -> /Batteries/BATT_VBUS
- C24 pad 1: /Batteries/BATT_VBUS -> Net-(U4-PMID)
- C25 pad 1: /Batteries/BATT_VBUS -> Net-(U4-PMID)
- C26 pad 1: /Batteries/BATT_VBUS -> Net-(U4-PMID)
- C27 pad 1: VBUS -> Net-(U4-BTST1)
- C27 pad 2: GND -> Net-(U4-SW1)
- C28 pad 1: Net-(U4-PMID) -> Net-(U4-BTST2)
- C28 pad 2: GND -> Net-(U4-SW2)
- C30 pad 1: Net-(U4-PMID) -> VBUS
- C31 pad 1: Net-(U4-PMID) -> VBUS
- C32 pad 1: Net-(U4-BTST1) -> VBUS
- C32 pad 2: Net-(U4-SW1) -> GND
- C33 pad 1: Net-(U4-BTST2) -> Net-(Q5-S)
- C33 pad 2: Net-(U4-SW2) -> GND
- C36 pad 1: VBUS -> Net-(Q5-S)
- C4 pad 1: VBUS -> /Batteries/USB_VIN
- C40 pad 1: /Batteries/REGN -> /Voltage Regulation/BOARD_LOAD_+
- C40 pad 2: Net-(C40-Pad2) -> GND
- C41 pad 1: Net-(C40-Pad2) -> +3V3
- C42 pad 1: Net-(U5-MR_N) -> +3V3
- C5 pad 1: /Voltage Regulation/BOARD_LOAD_+ -> /Batteries/EXTERNAL_VIN
- C6 pad 1: +3V3 -> Net-(U3-MR_N)
- D2 pad 2: /Batteries/REGN -> Net-(D2-A)
- J2 pad 1: /Batteries/EXTERNAL_VIN -> (no net)
- J2 pad 2: GND -> (no net)
- J5 pad 18: unconnected-(J5-Pad18) -> /System Bus/VSOLAR_1
- J5 pad 20: unconnected-(J5-Pad20) -> /System Bus/VSOLAR_2
- J5 pad 22: unconnected-(J5-Pad22) -> /System Bus/VSOLAR_3
- J5 pad 24: unconnected-(J5-Pad24) -> /System Bus/VSOLAR_4
- J5 pad 26: unconnected-(J5-Pad26) -> /System Bus/VSOLAR_5
- J5 pad 28: unconnected-(J5-Pad28) -> /System Bus/VSOLAR_6
- J5 pad 54: unconnected-(J5-Pad54) -> VBUS
- J5 pad 55: VBUS -> unconnected-(J5-Pad55)
- J5 pad 56: VBUS -> /CANH_UPSTREAM
- J5 pad 57: /CANH_UPSTREAM -> unconnected-(J5-Pad57)
- J6 pad 18: unconnected-(J6-Pad18) -> /System Bus/VSOLAR_1
- J6 pad 20: unconnected-(J6-Pad20) -> /System Bus/VSOLAR_2
- J6 pad 22: unconnected-(J6-Pad22) -> /System Bus/VSOLAR_3
- J6 pad 24: unconnected-(J6-Pad24) -> /System Bus/VSOLAR_4
- J6 pad 26: unconnected-(J6-Pad26) -> /System Bus/VSOLAR_5
- J6 pad 28: unconnected-(J6-Pad28) -> /System Bus/VSOLAR_6
- J6 pad 54: unconnected-(J6-Pad54) -> VBUS
- J6 pad 55: VBUS -> unconnected-(J6-Pad55)
- J6 pad 56: VBUS -> /CANH_DOWNSTREAM
- J6 pad 57: /CANH_DOWNSTREAM -> unconnected-(J6-Pad57)
- JP7 pad 2: Net-(JP7-B) -> /Batteries/REGN
- L1 pad 1: Net-(U8-LX2) -> Net-(U4-SW2)
- L1 pad 2: Net-(U8-LX1) -> Net-(U4-SW1)
- L2 pad 1: Net-(U4-SW2) -> Net-(U5-LX2)
- L2 pad 2: Net-(U4-SW1) -> Net-(U5-LX1)
- Q1 pad 1: Net-(D3-K) -> Net-(D2-K)
- Q1 pad 2: Net-(D3-A) -> Net-(D2-A)
- Q1 pad 3: /Batteries/USB_VIN -> /Batteries/EXTERNAL_VIN
- Q2 pad 3: /Batteries/BATT_VBUS -> /Batteries/USB_VIN
- Q3 pad 1: Net-(D4-K) (its old number) -> Net-(D2-K)
- Q3 pad 2: Net-(D4-A) -> Net-(D2-A)
- Q3 pad 3: /Batteries/EXTERNAL_VIN -> /Batteries/BATT_VBUS
- Q4 pad 1: Net-(D4-K) (its old number) -> Net-(D3-K)
- Q4 pad 2: Net-(D4-A) -> Net-(D3-A)
- R10 pad 1: /Voltage Regulation/BOARD_LOAD_+ -> Net-(U4-PROG)
- R10 pad 2: +3V3 -> GND
- R23 pad 1: Net-(U4-TS) -> Net-(U4-PROG)
- R24 pad 1: Net-(D2-K) -> Net-(JP8-A)
- R24 pad 2: Net-(U4-STAT) -> GND
- R25 pad 1: +3V3 -> Net-(D2-K)
- R25 pad 2: Net-(U3-SLOW) -> Net-(U4-ACDRV2)
- R26 pad 1: Net-(U4-BATP) -> Net-(JP7-A)
- R26 pad 2: /Batteries/VBATT -> Net-(JP12-B)
- R28 pad 1: Net-(D4-K) (its old number) -> Net-(JP12-A)
- R28 pad 2: Net-(U4-ACDRV2) -> GND
- R29 pad 1: Net-(U4-PROG) -> +3V3
- R29 pad 2: GND -> /Batteries/BATT_INT
- R30 pad 1: /Batteries/REGN -> Net-(JP11-A)
- R30 pad 2: Net-(U4-TS) -> Net-(JP12-B)
- R31 pad 1: Net-(U4-PROG) -> Net-(JP17-A)
- R32 pad 2: GND -> Net-(JP12-B)
- R33 pad 2: GND -> Net-(U4-STAT)
- R34 pad 1: +3V3 -> Net-(U4-BATP)
- R34 pad 2: /Batteries/BATT_INT -> /Batteries/VBATT
- R51 pad 1: Net-(U8-CFG1) -> Net-(J2-CC1)
- TH1 pad 1: Net-(U4-TS) -> Net-(JP8-A)
- TP1 pad 1: VBUS -> Net-(JP12-B)
- TP3 pad 1: GND -> VBUS
- U3 pad 1: Net-(U3-SLOW) -> Net-(JP9-A)
- U3 pad 2: +3V3 -> /Batteries/BATT_VBUS
- U3 pad 4: /Batteries/I2C_SDA -> Net-(U3-MR_N)
- U3 pad 5: /Batteries/I2C_SCL -> Net-(U3-CT)
- U4 pad 12: Net-(JP7-B) -> Net-(JP9-B)
- U4 pad 16: Net-(U4-TS) -> Net-(JP12-B)
- U5 pad 1: Net-(JP7-A) -> VBUS
- U5 pad 2: /Batteries/BATT_VBUS -> VBUS
- U5 pad 3: GND -> Net-(U5-CFG1)
- U5 pad 4: Net-(U5-MR_N) -> GND
- U5 pad 5: Net-(U5-CT) -> GND
- U8 pad 1: VBUS -> Net-(U8-SLOW)
- U8 pad 10: VBUS -> unconnected-(U8-SENSE4+-Pad10)
- U8 pad 11: GND -> /Voltage Regulation/BOARD_LOAD_+
- U8 pad 2: VBUS -> +3V3
- U8 pad 3: Net-(U8-CFG1) -> GND
- U8 pad 4: GND -> /Batteries/I2C_SCL
- U8 pad 5: GND -> /Batteries/I2C_SDA
- U8 pad 6: /Voltage Regulation/BOARD_LOAD_+ -> GND
- U8 pad 7: Net-(U8-LX2) -> unconnected-(U8-SENSE3--Pad7)
- U8 pad 8: GND -> unconnected-(U8-SENSE3+-Pad8)
- U8 pad 9: Net-(U8-LX1) -> unconnected-(U8-SENSE4--Pad9)
Routing:
- net +3V3: track 32.2 -> 29.4 mm, vias 21 -> 19
- net Net-(U3-MR_N): track 0.00 -> 2.03 mm, vias 0 -> 2
- net Net-(U4-ACDRV2): track 0.00 -> 1.50 mm
- net Net-(U3-SLOW): track 1.50 -> 0.00 mm
- net Net-(D2-K): track 0.00 -> 0.79 mm, vias 0 -> 1
- net Net-(C17-Pad2): track 0.00 -> 0.77 mm
- net GND: track 55.1 -> 54.4 mm, vias 36 -> 32
- net Net-(U3-CT): vias 0 -> 1
- net Net-(JP9-A): vias 0 -> 1

Commit message: Add hierarchical sheet and PCB layout for the core board, including the system bus.
Parts:
- removed BT1, BT2, BT3: Battery_Cell, footprints:BAT_1043
- removed C1, C13, C14, C2, C23, C24, C3, C30, C4, C41, C42, C5, C6, C7, C8, C9: 100n, footprints:Nondescript_C_0402_1005Metric
- removed C10, C11, C12, C15, C16: 1u, footprints:Nondescript_C_0402_1005Metric
- removed C17, C18, C21, C22, C25, C26, C29, C31, C32, C33, C34, C35, C36, C37, C39: 10u, footprints:Nondescript_C_0603_1608Metric
- removed C19: 1n, footprints:Nondescript_C_0603_1608Metric
- removed C27, C28: 0.047u, footprints:Nondescript_C_0402_1005Metric
- removed C38, C40: 22u, footprints:Nondescript_C_0603_1608Metric
- removed D1, D4: Blue LED, LED_SMD:LED_0603_1608Metric
- removed D2: Zener, LED_SMD:LED_0603_1608Metric
- removed J1: STLINK, Connector:Tag-Connect_TC2030-IDC-NL_2x03_P1.27mm_Vertical
- removed J2: USB_C_Receptacle, footprints:B2BPHKSLFSN
- removed J5: QTH-030-07-L-D-A, footprints:SAMTEC_QTH-030-07-L-D-A
- removed J6: QSH-030-01-L-D-A, footprints:SAMTEC_QSH-030-01-L-D-A
- removed JP1, JP10, JP11, JP12, JP13, JP16, JP17, JP2, JP3, JP4, JP5, JP6, JP7, JP8, JP9: SolderJumper_2_Open, Jumper:SolderJumper-2_P1.3mm_Open_RoundedPad1.0x1.5mm
- removed JP14: 0x10, Jumper:SolderJumper-2_P1.3mm_Open_RoundedPad1.0x1.5mm
- removed JP15: 0xEF, Jumper:SolderJumper-2_P1.3mm_Open_RoundedPad1.0x1.5mm
- removed L1, L2, L3, L4, L5, L6, L7, L8: 2.2µH, Inductor_SMD:L_1008_2520Metric
- removed PCB1: ~, footprints:Core_Board
- removed Q1, Q2, Q3, Q4, Q5: CSD13385F5, footprints:PICOSTAR3_YJK_TEX
- removed R1, R10, R13, R14, R23, R29, R3, R40, R42, R45, R48, R54, R57, R6, R60: 9k31, footprints:Nondescript_R_0402_1005Metric
- removed R17, R22: 23k2, footprints:Nondescript_R_0402_1005Metric
- removed R2, R33, R37, R38, R39, R4, R5, R7, R8, R9: 33, footprints:Nondescript_R_0402_1005Metric
- removed R20, R21: 1k58, footprints:Nondescript_R_0402_1005Metric
- removed R24, R28, R31: 57k9, footprints:Nondescript_R_0402_1005Metric
- removed R25, R27: 294, Resistor_SMD:R_0402_1005Metric_Pad0.72x0.64mm_HandSolder
- removed R26, R30, R32: 7k2, footprints:Nondescript_R_0402_1005Metric
- removed R34: 100, Resistor_SMD:R_0402_1005Metric_Pad0.72x0.64mm_HandSolder
- removed R35: 36k5, footprints:Nondescript_R_0402_1005Metric
- removed R36: 100m, Resistor_SMD:R_0805_2012Metric
- removed R41, R51: 5k1, Resistor_SMD:R_0402_1005Metric_Pad0.72x0.64mm_HandSolder
- removed R49, R50: 60, footprints:Nondescript_R_0402_1005Metric
- removed TH1, TH2, TH3: 10k NTC, footprints:Nondescript_R_0603_1608Metric
- removed TP1: TEMP, footprints:TestPoint_Pad_D1.5mm
- removed TP2: BOARD_ID_POWER, footprints:TestPoint_Pad_D1.5mm
- removed TP3: VBUS, footprints:TestPoint_Pad_D1.5mm
- removed TP5: BOARD_ID_SENSE, footprints:TestPoint_Pad_D1.5mm
- removed U1: STM32L452RCTx, Package_QFP:LQFP-64_10x10mm_P0.5mm
- removed U10, U11, U14, U16, U18, U7: SPV1040TTR, footprints:SOIC_1040T_STM
- removed U12, U13, U15, U17, U6, U9: LM66100DCK, Package_TO_SOT_SMD:SOT-363_SC-70-6
- removed U2: TCAN330DR, footprints:SOIC127P600X175-8N
- removed U3: TPS3840DL18DBVR, footprints:DBV0005A_L
- removed U4: BQ25798, Package_DFN_QFN:Texas_RQM0029A_VQFN-29_4x4mm_P0.4mm
- removed U5: TPS63900, Package_SON:WSON-10-1EP_2.5x2.5mm_P0.5mm_EP1.2x2mm_ThermalVias
- removed U8: PAC1934T-I/JQ, Package_DFN_QFN:UQFN-16-1EP_4x4mm_P0.65mm_EP2.6x2.6mm
- added BT801: Battery_Cell, footprints:BAT_1043, F.Cu at (134.8, 104.9)
- added BT802: Battery_Cell, footprints:BAT_1043, F.Cu at (156.0, 104.9)
- added BT803: Battery_Cell, footprints:BAT_1043, F.Cu at (177.2, 104.9)
- added C201: 100n, footprints:Nondescript_C_0402_1005Metric, F.Cu at (35.0, 131.7)
- added C202: 100n, footprints:Nondescript_C_0402_1005Metric, F.Cu at (35.0, 133.7)
- added C203: 1u, footprints:Nondescript_C_0402_1005Metric, F.Cu at (35.0, 135.6)
- added C204: 100n, footprints:Nondescript_C_0402_1005Metric, F.Cu at (35.0, 137.6)
- added C205: 1u, footprints:Nondescript_C_0402_1005Metric, F.Cu at (35.0, 139.6)
- added C206: 100n, footprints:Nondescript_C_0402_1005Metric, F.Cu at (37.9, 131.7)
- added C207: 100n, footprints:Nondescript_C_0402_1005Metric, F.Cu at (37.9, 133.7)
- added C208: 1u, footprints:Nondescript_C_0402_1005Metric, F.Cu at (37.9, 135.6)
- added C209: 100n, footprints:Nondescript_C_0402_1005Metric, F.Cu at (37.9, 137.6)
- added C210: 1u, footprints:Nondescript_C_0402_1005Metric, F.Cu at (37.9, 139.6)
- added C601: 1u, footprints:Nondescript_C_0402_1005Metric, F.Cu at (39.3, 171.5)
- added C602: 100n, footprints:Nondescript_C_0402_1005Metric, F.Cu at (39.3, 173.4)
- added C603: 100n, footprints:Nondescript_C_0402_1005Metric, F.Cu at (39.3, 175.4)
- added C701: 22u, footprints:Nondescript_C_0603_1608Metric, F.Cu at (36.4, 31.7)
- added C702: 10u, footprints:Nondescript_C_0603_1608Metric, F.Cu at (36.4, 34.2)
- added C703: 22u, footprints:Nondescript_C_0603_1608Metric, F.Cu at (36.4, 36.8)
- added C704: 100n, footprints:Nondescript_C_0402_1005Metric, F.Cu at (46.4, 31.5)
- added C705: 100n, footprints:Nondescript_C_0402_1005Metric, F.Cu at (46.4, 33.4)
- added C801: 100n, footprints:Nondescript_C_0402_1005Metric, F.Cu at (28.6, 142.1)
- added C802: 100n, footprints:Nondescript_C_0402_1005Metric, F.Cu at (28.6, 144.1)
- added C803: 100n, footprints:Nondescript_C_0402_1005Metric, F.Cu at (28.6, 146.0)
- added C804: 10u, footprints:Nondescript_C_0603_1608Metric, F.Cu at (-49.4, 184.1)
- added C805: 10u, footprints:Nondescript_C_0603_1608Metric, F.Cu at (-49.4, 186.6)
- added C808: 10u, footprints:Nondescript_C_0603_1608Metric, F.Cu at (-49.4, 189.1)
- added C809: 10u, footprints:Nondescript_C_0603_1608Metric, F.Cu at (-49.4, 191.6)
- added C810: 100n, footprints:Nondescript_C_0402_1005Metric, F.Cu at (28.6, 148.0)
- added C811: 100n, footprints:Nondescript_C_0402_1005Metric, F.Cu at (28.6, 150.0)
- added C812: 10u, footprints:Nondescript_C_0603_1608Metric, F.Cu at (-49.4, 194.1)
- added C813: 10u, footprints:Nondescript_C_0603_1608Metric, F.Cu at (-49.4, 196.7)
- added C814: 0.047u, footprints:Nondescript_C_0402_1005Metric, F.Cu at (28.6, 151.9)
- added C815: 0.047u, footprints:Nondescript_C_0402_1005Metric, F.Cu at (28.6, 153.9)
- added C816: 10u, footprints:Nondescript_C_0603_1608Metric, F.Cu at (-45.4, 184.1)
- added C817: 100n, footprints:Nondescript_C_0402_1005Metric, F.Cu at (28.6, 155.9)
- added C818: 10u, footprints:Nondescript_C_0603_1608Metric, F.Cu at (-45.4, 186.6)
- added C819: 10u, footprints:Nondescript_C_0603_1608Metric, F.Cu at (-45.4, 189.1)
- added C820: 10u, footprints:Nondescript_C_0603_1608Metric, F.Cu at (-45.4, 191.6)
- added C821: 10u, footprints:Nondescript_C_0603_1608Metric, F.Cu at (-45.4, 194.1)
- added C822: 10u, footprints:Nondescript_C_0603_1608Metric, F.Cu at (-45.4, 196.7)
- added C823: 10u, footprints:Nondescript_C_0603_1608Metric, F.Cu at (-41.4, 184.1)
- added C824: 10u, footprints:Nondescript_C_0603_1608Metric, F.Cu at (-41.4, 186.6)
- added D201: Blue LED, LED_SMD:LED_0603_1608Metric, F.Cu at (41.3, 132.0)
- added D803: Blue LED, LED_SMD:LED_0603_1608Metric, F.Cu at (-22.0, 192.2)
- added J401: STLINK, Connector:Tag-Connect_TC2030-IDC-NL_2x03_P1.27mm_Vertical, F.Cu at (41.3, 49.0)
- added J501: QTH-030-07-L-D-A, footprints:SAMTEC_QTH-030-07-L-D-A, F.Cu at (119.7, 127.0)
- added J502: QSH-030-01-L-D-A, footprints:SAMTEC_QSH-030-01-L-D-A, B.Cu at (119.7, 127.0)
- added JP301: SolderJumper_2_Open, Jumper:SolderJumper-2_P1.3mm_Open_RoundedPad1.0x1.5mm, F.Cu at (50.6, 165.7)
- added JP302: SolderJumper_2_Open, Jumper:SolderJumper-2_P1.3mm_Open_RoundedPad1.0x1.5mm, F.Cu at (50.6, 169.3)
- added JP303: 0x10, Jumper:SolderJumper-2_P1.3mm_Open_RoundedPad1.0x1.5mm, F.Cu at (50.6, 172.8)
- added JP304: 0xEF, Jumper:SolderJumper-2_P1.3mm_Open_RoundedPad1.0x1.5mm, F.Cu at (50.6, 176.4)
- added JP601: SolderJumper_2_Open, Jumper:SolderJumper-2_P1.3mm_Open_RoundedPad1.0x1.5mm, F.Cu at (35.7, 165.7)
- added JP602: SolderJumper_2_Open, Jumper:SolderJumper-2_P1.3mm_Open_RoundedPad1.0x1.5mm, F.Cu at (35.7, 169.3)
- added JP603: SolderJumper_2_Open, Jumper:SolderJumper-2_P1.3mm_Open_RoundedPad1.0x1.5mm, F.Cu at (35.7, 172.8)
- added JP604: SolderJumper_2_Open, Jumper:SolderJumper-2_P1.3mm_Open_RoundedPad1.0x1.5mm, F.Cu at (35.7, 176.4)
- added JP605: SolderJumper_2_Open, Jumper:SolderJumper-2_P1.3mm_Open_RoundedPad1.0x1.5mm, F.Cu at (35.7, 179.9)
- added JP606: SolderJumper_2_Open, Jumper:SolderJumper-2_P1.3mm_Open_RoundedPad1.0x1.5mm, F.Cu at (35.7, 183.5)
- added JP801: SolderJumper_2_Open, Jumper:SolderJumper-2_P1.3mm_Open_RoundedPad1.0x1.5mm, F.Cu at (29.4, 118.0)
- added JP802: SolderJumper_2_Open, Jumper:SolderJumper-2_P1.3mm_Open_RoundedPad1.0x1.5mm, F.Cu at (29.4, 121.6)
- added JP803: SolderJumper_2_Open, Jumper:SolderJumper-2_P1.3mm_Open_RoundedPad1.0x1.5mm, F.Cu at (29.4, 125.1)
- added JP804: SolderJumper_2_Open, Jumper:SolderJumper-2_P1.3mm_Open_RoundedPad1.0x1.5mm, F.Cu at (29.4, 128.7)
- added JP805: SolderJumper_2_Open, Jumper:SolderJumper-2_P1.3mm_Open_RoundedPad1.0x1.5mm, F.Cu at (29.4, 132.2)
- added JP806: SolderJumper_2_Open, Jumper:SolderJumper-2_P1.3mm_Open_RoundedPad1.0x1.5mm, F.Cu at (29.4, 135.8)
- added JP807: SolderJumper_2_Open, Jumper:SolderJumper-2_P1.3mm_Open_RoundedPad1.0x1.5mm, F.Cu at (29.4, 139.3)
- added L1101: 2.2µH, Inductor_SMD:L_1008_2520Metric, F.Cu at (36.8, 85.9)
- added L1201: 2.2µH, Inductor_SMD:L_1008_2520Metric, F.Cu at (48.4, 61.1)
- added L1301: 2.2µH, Inductor_SMD:L_1008_2520Metric, F.Cu at (36.8, 61.1)
- added L1401: 2.2µH, Inductor_SMD:L_1008_2520Metric, F.Cu at (48.4, 73.5)
- added L1501: 2.2µH, Inductor_SMD:L_1008_2520Metric, F.Cu at (36.8, 73.5)
- added L1601: 2.2µH, Inductor_SMD:L_1008_2520Metric, F.Cu at (48.4, 85.9)
- added L701: 2.2µH, Inductor_SMD:L_1008_2520Metric, F.Cu at (40.9, 42.6)
- added L801: 2.2µH, Inductor_SMD:L_1008_2520Metric, F.Cu at (-21.6, 184.7)
- added PCB101: ~, footprints:Core_Board, F.Cu at (114.7, 146.2)
- added Q801: CSD13385F5, footprints:PICOSTAR3_YJK_TEX, F.Cu at (-37.8, 184.1)
- added Q802: CSD13385F5, footprints:PICOSTAR3_YJK_TEX, F.Cu at (-37.8, 186.5)
- added Q803: CSD13385F5, footprints:PICOSTAR3_YJK_TEX, F.Cu at (-37.8, 188.9)
- added Q804: CSD13385F5, footprints:PICOSTAR3_YJK_TEX, F.Cu at (-37.8, 191.3)
- added Q805: CSD13385F5, footprints:PICOSTAR3_YJK_TEX, F.Cu at (-37.8, 193.7)
- added R1101: 9k31, footprints:Nondescript_R_0402_1005Metric, F.Cu at (40.8, 88.6)
- added R1201: 9k31, footprints:Nondescript_R_0402_1005Metric, F.Cu at (52.4, 63.9)
- added R1301: 9k31, footprints:Nondescript_R_0402_1005Metric, F.Cu at (40.8, 63.9)
- added R1401: 9k31, footprints:Nondescript_R_0402_1005Metric, F.Cu at (52.4, 76.3)
- added R1501: 9k31, footprints:Nondescript_R_0402_1005Metric, F.Cu at (40.8, 76.3)
- added R1601: 9k31, footprints:Nondescript_R_0402_1005Metric, F.Cu at (52.4, 88.6)
- added R201: 33, footprints:Nondescript_R_0402_1005Metric, F.Cu at (49.5, 117.2)
- added R205: 9k31, footprints:Nondescript_R_0402_1005Metric, F.Cu at (49.5, 119.2)
- added R206: 9k31, footprints:Nondescript_R_0402_1005Metric, F.Cu at (49.5, 121.2)
- added R208: 33, footprints:Nondescript_R_0402_1005Metric, F.Cu at (49.5, 123.2)
- added R209: 33, footprints:Nondescript_R_0402_1005Metric, F.Cu at (49.5, 125.2)
- added R210: 33, footprints:Nondescript_R_0402_1005Metric, F.Cu at (49.5, 127.2)
- added R211: 33, footprints:Nondescript_R_0402_1005Metric, F.Cu at (52.4, 117.2)
- added R212: 9k31, footprints:Nondescript_R_0402_1005Metric, F.Cu at (52.4, 119.2)
- added R214: 9k31, footprints:Nondescript_R_0402_1005Metric, F.Cu at (52.4, 121.2)
- added R215: 9k31, footprints:Nondescript_R_0402_1005Metric, F.Cu at (52.4, 123.2)
- added R216: 33, footprints:Nondescript_R_0402_1005Metric, F.Cu at (52.4, 125.2)
- added R301: 23k2, footprints:Nondescript_R_0402_1005Metric, F.Cu at (54.2, 172.0)
- added R302: 1k58, footprints:Nondescript_R_0402_1005Metric, F.Cu at (54.2, 174.0)
- added R303: 1k58, footprints:Nondescript_R_0402_1005Metric, F.Cu at (54.2, 176.0)
- added R304: 23k2, footprints:Nondescript_R_0402_1005Metric, F.Cu at (54.2, 178.0)
- added R401: 33, footprints:Nondescript_R_0402_1005Metric, F.Cu at (35.8, 47.5)
- added R402: 33, footprints:Nondescript_R_0402_1005Metric, F.Cu at (35.8, 49.5)
- added R403: 33, footprints:Nondescript_R_0402_1005Metric, F.Cu at (35.8, 51.5)
- added R601: 60, footprints:Nondescript_R_0402_1005Metric, F.Cu at (42.2, 171.5)
- added R602: 60, footprints:Nondescript_R_0402_1005Metric, F.Cu at (42.2, 173.5)
- added R701: 36k5, footprints:Nondescript_R_0402_1005Metric, F.Cu at (45.0, 40.7)
- added R702: 100m, Resistor_SMD:R_0805_2012Metric, F.Cu at (45.8, 38.2)
- added R703: 9k31, footprints:Nondescript_R_0402_1005Metric, F.Cu at (45.0, 42.7)
- added R801: 9k31, footprints:Nondescript_R_0402_1005Metric, F.Cu at (-34.7, 183.8)
- added R802: 9k31, footprints:Nondescript_R_0402_1005Metric, F.Cu at (-34.7, 185.8)
- added R803: 57k9, footprints:Nondescript_R_0402_1005Metric, F.Cu at (-34.7, 187.8)
- added R804: 294, Resistor_SMD:R_0402_1005Metric_Pad0.72x0.64mm_HandSolder, F.Cu at (-28.7, 189.8)
- added R805: 7k2, footprints:Nondescript_R_0402_1005Metric, F.Cu at (-34.7, 189.8)
- added R806: 294, Resistor_SMD:R_0402_1005Metric_Pad0.72x0.64mm_HandSolder, F.Cu at (-28.7, 191.8)
- added R807: 57k9, footprints:Nondescript_R_0402_1005Metric, F.Cu at (-34.7, 191.8)
- added R808: 9k31, footprints:Nondescript_R_0402_1005Metric, F.Cu at (-31.8, 183.8)
- added R809: 7k2, footprints:Nondescript_R_0402_1005Metric, F.Cu at (-31.8, 185.8)
- added R810: 57k9, footprints:Nondescript_R_0402_1005Metric, F.Cu at (-31.8, 187.8)
- added R811: 7k2, footprints:Nondescript_R_0402_1005Metric, F.Cu at (-31.8, 189.8)
- added R812: 33, footprints:Nondescript_R_0402_1005Metric, F.Cu at (-31.8, 191.8)
- added R813: 100, Resistor_SMD:R_0402_1005Metric_Pad0.72x0.64mm_HandSolder, F.Cu at (-28.7, 193.8)
- added R901: 5k1, Resistor_SMD:R_0402_1005Metric_Pad0.72x0.64mm_HandSolder, F.Cu at (36.0, 92.6)
- added R902: 5k1, Resistor_SMD:R_0402_1005Metric_Pad0.72x0.64mm_HandSolder, F.Cu at (36.0, 94.6)
- added TH801: 10k NTC, footprints:Nondescript_R_0603_1608Metric, F.Cu at (-41.4, 189.1)
- added TH802: 10k NTC, footprints:Nondescript_R_0603_1608Metric, F.Cu at (-41.4, 191.6)
- added TH803: 10k NTC, footprints:Nondescript_R_0603_1608Metric, F.Cu at (-41.4, 194.1)
- added TP301: BOARD_ID_SENSE, footprints:TestPoint_Pad_D1.5mm, F.Cu at (54.5, 165.7)
- added TP302: BOARD_ID_POWER, footprints:TestPoint_Pad_D1.5mm, F.Cu at (54.5, 169.3)
- added TP701: VBUS, footprints:TestPoint_Pad_D1.5mm, F.Cu at (36.1, 39.8)
- added TP801: TEMP, footprints:TestPoint_Pad_D1.5mm, F.Cu at (-22.3, 195.3)
- added U1101: LM66100DCK, Package_TO_SOT_SMD:SOT-363_SC-70-6, F.Cu at (41.6, 85.9)
- added U1102: SPV1040TTR, footprints:SOIC_1040T_STM, F.Cu at (38.8, 81.6)
- added U1201: LM66100DCK, Package_TO_SOT_SMD:SOT-363_SC-70-6, F.Cu at (53.2, 61.1)
- added U1202: SPV1040TTR, footprints:SOIC_1040T_STM, F.Cu at (50.4, 56.9)
- added U1301: LM66100DCK, Package_TO_SOT_SMD:SOT-363_SC-70-6, F.Cu at (41.6, 61.1)
- added U1302: SPV1040TTR, footprints:SOIC_1040T_STM, F.Cu at (38.8, 56.9)
- added U1401: LM66100DCK, Package_TO_SOT_SMD:SOT-363_SC-70-6, F.Cu at (53.2, 73.5)
- added U1402: SPV1040TTR, footprints:SOIC_1040T_STM, F.Cu at (50.4, 69.3)
- added U1501: LM66100DCK, Package_TO_SOT_SMD:SOT-363_SC-70-6, F.Cu at (41.6, 73.5)
- added U1502: SPV1040TTR, footprints:SOIC_1040T_STM, F.Cu at (38.8, 69.3)
- added U1601: LM66100DCK, Package_TO_SOT_SMD:SOT-363_SC-70-6, F.Cu at (53.2, 85.9)
- added U1602: SPV1040TTR, footprints:SOIC_1040T_STM, F.Cu at (50.4, 81.6)
- added U201: STM32L452RCTx, Package_QFP:LQFP-64_10x10mm_P0.5mm, F.Cu at (40.8, 123.5)
- added U601: TCAN330DR, footprints:SOIC127P600X175-8N, F.Cu at (42.1, 167.2)
- added U701: TPS63900, Package_SON:WSON-10-1EP_2.5x2.5mm_P0.5mm_EP1.2x2mm_ThermalVias, F.Cu at (41.2, 38.8)
- added U702: PAC1934T-I/JQ, Package_DFN_QFN:UQFN-16-1EP_4x4mm_P0.65mm_EP2.6x2.6mm, F.Cu at (41.9, 33.6)
- added U801: TPS3840DL18DBVR, footprints:DBV0005A_L, F.Cu at (-21.8, 188.8)
- added U802: BQ25798, Package_DFN_QFN:Texas_RQM0029A_VQFN-29_4x4mm_P0.4mm, F.Cu at (-27.0, 185.8)
Routing:
- net GND: track 54.4 -> 0.00 mm, vias 32 -> 0
- net /SWDIO: track 48.9 -> 0.00 mm, vias 1 -> 0
- net /SWO: track 44.2 -> 0.00 mm, vias 1 -> 0
- net /MCU/DEBUG_LED: track 42.6 -> 0.00 mm, vias 2 -> 0
- net /SWCLK: track 41.3 -> 0.00 mm
- net /NRST: track 32.7 -> 0.00 mm
- net +3V3: track 29.4 -> 0.00 mm, vias 19 -> 0
- net /CAN bus/CAN_SILENT: track 28.3 -> 0.00 mm
- net /CAN bus/CAN_SHUTDOWN: track 28.2 -> 0.00 mm
- net Net-(JP1-B): track 25.9 -> 0.00 mm, vias 2 -> 0
- net Net-(JP2-B): track 23.0 -> 0.00 mm
- net /CAN bus/CAN_TX: track 22.4 -> 0.00 mm
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- removed copper zone on B.Cu, net +3V3
- removed copper zone on In2.Cu, net +3V3
- removed copper zone on B.Cu, net /Voltage Regulation/BOARD_LOAD_+
- removed copper zone on B.Cu, net GND
- removed copper zone on B.Cu, net VBUS
Other:
- board text removed: "Board ID"
- board text removed: "CAN Termination"
- board text removed: "Downstream CAN"
- board text removed: "Upstream CAN"
