File: electrical/pcb_design/1s3p_battery_board/power.kicad_sch (KiCad schematic)
At the start: 11 parts, among them U8 TPS63900

Commit message: Move 1s3p battery board to KiCad 9
Changed lines of the file:
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@@
 (kicad_sch
-	(version 20231120)
+	(version 20250114)
 	(generator "eeschema")
-	(generator_version "8.0")
+	(generator_version "9.0")
 	(paper "USLetter")
 	(title_block
@@
 		)
 		(instances
-			(project ""
+			(project "1s3p_battery_board"
 				(path "/695f882b-5312-4493-b26d-8f7d6768a9db/7f8fc7f5-7f1e-476b-9e93-5575de1d6778"
 					(reference "L1")
@@
 		)
 		(instances
-			(project ""
+			(project "1s3p_battery_board"
 				(path "/695f882b-5312-4493-b26d-8f7d6768a9db/7f8fc7f5-7f1e-476b-9e93-5575de1d6778"
 					(reference "U8")

Commit message: Checkpoint work on 1s3p battery board
Parts:
- added C17, C6: 100n, footprints:Nondescript_C_0402_1005Metric, symbol Device:C
- added R25: 9k31, footprints:Nondescript_R_0402_1005Metric, symbol Device:R_Small
- added U3: PAC1934T-I/JQ, footprints:UQFN-16-1EP_4x4mm_P0.65mm_EP2.6x2.6mm, symbol Sensor_Energy:PAC1934x-xJQ
Connections:
- net +3V3: now also C17.1, C6.1, R25.1, U3.14 (SENSE2-), U3.15 (V_{DD}IO), U3.16 (~{PWRDN}), U3.2 (V_{DD})
- net BOARD_LOAD_+: now also U3.13 (SENSE2+)
- net GND: now also C17.2, C6.2, U3.17 (EP), U3.3 (GND), U3.6 (ADDRSEL)
- new net: R25.2, U3.1 (SLOW)
- new net I2C_SCL: U3.4 (SCL)
- new net I2C_SDA: U3.5 (SDA)
- no-connect marks 0 -> 6
Other:
- note added: "Board Power Monitor"
- moved on the sheet: C27, C4, C5, L1, R10, R51, TP1, TP3, TP4, TP6, U8

Commit message: Restructure battery board with new system bus, power monitoring chip, and battery charging IC.
Parts:
- U3: footprint footprints:UQFN-16-1EP_4x4mm_P0.65mm_EP2.6x2.6mm -> Package_DFN_QFN:UQFN-16-1EP_4x4mm_P0.65mm_EP2.6x2.6mm
- U8: footprint Package_SON:WSON-10-1EP_2.5x2.5mm_P0.5mm_EP1.2x2mm -> Package_SON:WSON-10-1EP_2.5x2.5mm_P0.5mm_EP1.2x2mm_ThermalVias
Connections:
- net BOARD_LOAD_+: now also U3.11 (SENSE1+); no longer U3.13 (SENSE2+)
- net 3V3: now reaches U3.12 (SENSE1-)
- net 3V3: now also C17.1, C6.1, R10.2, R25.1, TP6.1, U3.15 (V_{DD}IO), U3.16 (~{PWRDN}), U3.2 (V_{DD})
- removed net +3V3: C17.1, C6.1, R10.2, R25.1, TP6.1, U3.14 (SENSE2-), U3.15 (V_{DD}IO), U3.16 (~{PWRDN}), U3.2 (V_{DD})
Other:
- moved on the sheet: C17, C6, R25, U3

Commit message: Checkpoint work on 1s3p battery board.
Parts:
- removed TP4: BOARD_LOAD_+, footprints:TestPoint_Pad_D1.5mm, symbol Connector:TestPoint_Probe
- removed TP6: +3V3, footprints:TestPoint_Pad_D1.5mm, symbol Connector:TestPoint_Probe
- R10: value 10m -> 100m; footprint Resistor_SMD:R_2512_6332Metric -> Resistor_SMD:R_0805_2012Metric; Basic or Extended Component Extended -> Basic; MPN C241862 -> C1518131; Manufacturer Part Number WSLP2512R0100FEA -> WSL0805R1000DEA18
- R51: footprint footprints:Nondescript_R_0603_1608Metric -> footprints:Nondescript_R_0402_1005Metric; Basic or Extended Component Extended -> Basic; MPN C23029 -> C25887; Manufacturer Part Number 0603WAF3652T5E -> 0402WGF3652TCE

Commit message: Checkpoint progress on battery board. Preparing to break out reusable functional modules.
Parts:
- removed TP3: GND, footprints:TestPoint_Pad_D1.5mm, symbol Connector:TestPoint_Probe
- renumbered C27 to C38, C4 to C39, C5 to C40, C6 to C41, C17 to C42, L1 to L2, R51 to R35, R10 to R36, R25 to R40, TP1 to TP3, U8 to U5, U3 to U8
Changed lines of the file:
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@@
 		(on_board yes)
 		(dnp no)
-		(property "Reference" "L1"
+		(property "Reference" "L2"
 			(at 76.2 55.8799 0)
 			(effects
@@
 		(instances
 			(project "1s3p_battery_board"
-				(path "/695f882b-5312-4493-b26d-8f7d6768a9db/7f8fc7f5-7f1e-476b-9e93-5575de1d6778"
-					(reference "L1")
+				(path "/695f882b-5312-4493-b26d-8f7d6768a9db/64470299-6c65-479c-8ce7-e6a986c7fce1"
+					(reference "L2")
 					(unit 1)
 				)
@@
 		(on_board yes)
 		(dnp no)
-		(property "Reference" "U8"
+		(property "Reference" "U5"
 			(at 88.9 34.29 0)
 			(effects
@@
 		(instances
 			(project "1s3p_battery_board"
-				(path "/695f882b-5312-4493-b26d-8f7d6768a9db/7f8fc7f5-7f1e-476b-9e93-5575de1d6778"
-					(reference "U8")
+				(path "/695f882b-5312-4493-b26d-8f7d6768a9db/64470299-6c65-479c-8ce7-e6a986c7fce1"
+					(reference "U5")
 					(unit 1)
 				)
@@
 		(on_board yes)
 		(dnp no)
-		(property "Reference" "R51"
+		(property "Reference" "R35"
 			(at 102.87 46.99 90)
 			(effects
@@
 		(instances
 			(project "1s3p_battery_board"
-				(path "/695f882b-5312-4493-b26d-8f7d6768a9db/7f8fc7f5-7f1e-476b-9e93-5575de1d6778"
-					(reference "R51")
+				(path "/695f882b-5312-4493-b26d-8f7d6768a9db/64470299-6c65-479c-8ce7-e6a986c7fce1"
+					(reference "R35")
 					(unit 1)
 				)
@@
 		(on_board yes)
 		(dnp no)
-		(property "Reference" "U3"
+		(property "Reference" "U8"
 			(at 209.804 110.236 0)
 			(effects
@@
 		(instances
 			(project "1s3p_battery_board"
-				(path "/695f882b-5312-4493-b26d-8f7d6768a9db/7f8fc7f5-7f1e-476b-9e93-5575de1d6778"
-					(reference "U3")
+				(path "/695f882b-5312-4493-b26d-8f7d6768a9db/64470299-6c65-479c-8ce7-e6a986c7fce1"
+					(reference "U8")
 					(unit 1)
 				)
@@
 		(on_board yes)
 		(dnp no)
-		(property "Reference" "TP1"
+		(property "Reference" "TP3"
 			(at 64.77 39.0525 0)
 			(effects
@@
 		(instances
 			(project "1s3p_battery_board"
-				(path "/695f882b-5312-4493-b26d-8f7d6768a9db/7f8fc7f5-7f1e-476b-9e93-5575de1d6778"
-					(reference "TP1")
+				(path "/695f882b-5312-4493-b26d-8f7d6768a9db/64470299-6c65-479c-8ce7-e6a986c7fce1"
+					(reference "TP3")
 					(unit 1)
 				)
@@
 		(on_board yes)
 		(dnp no)
-		(property "Reference" "#PWR41"
+		(property "Reference" "#PWR048"
 			(at 173.99 82.55 0)
 			(effects
@@
 		(instances
 			(project "1s3p_battery_board"
-				(path "/695f882b-5312-4493-b26d-8f7d6768a9db/7f8fc7f5-7f1e-476b-9e93-5575de1d6778"
-					(reference "#PWR41")
+				(path "/695f882b-5312-4493-b26d-8f7d6768a9db/64470299-6c65-479c-8ce7-e6a986c7fce1"
+					(reference "#PWR048")
 					(unit 1)
 				)
@@
 		(on_board yes)
 		(dnp no)
-		(property "Reference" "C17"
+		(property "Reference" "C42"
 			(at 195.58 71.12 0)
 			(effects
@@
 		(instances
 			(project "1s3p_battery_board"
-				(path "/695f882b-5312-4493-b26d-8f7d6768a9db/7f8fc7f5-7f1e-476b-9e93-5575de1d6778"
-					(reference "C17")
+				(path "/695f882b-5312-4493-b26d-8f7d6768a9db/64470299-6c65-479c-8ce7-e6a986c7fce1"
+					(reference "C42")
 					(unit 1)
 				)
@@
 		(dnp no)
 		(fields_autoplaced yes)
-		(property "Reference" "R25"
+		(property "Reference" "R40"
 			(at 213.36 95.2499 0)
 			(effects
@@
 		(instances
 			(project "1s3p_battery_board"
-				(path "/695f882b-5312-4493-b26d-8f7d6768a9db/7f8fc7f5-7f1e-476b-9e93-5575de1d6778"
-					(reference "R25")
+				(path "/695f882b-5312-4493-b26d-8f7d6768a9db/64470299-6c65-479c-8ce7-e6a986c7fce1"
+					(reference "R40")
 					(unit 1)
 				)
@@
 		(on_board yes)
 		(dnp no)
-		(property "Reference" "#PWR33"
+		(property "Reference" "#PWR051"
 			(at 191.77 82.55 0)
 			(effects
@@
 		(instances
 			(project "1s3p_battery_board"
-				(path "/695f882b-5312-4493-b26d-8f7d6768a9db/7f8fc7f5-7f1e-476b-9e93-5575de1d6778"
-					(reference "#PWR33")
+				(path "/695f882b-5312-4493-b26d-8f7d6768a9db/64470299-6c65-479c-8ce7-e6a986c7fce1"
+					(reference "#PWR051")
 					(unit 1)
 				)
@@
 		(on_board yes)
 		(dnp no)
-		(property "Reference" "R10"
+		(property "Reference" "R36"
 			(at 140.335 45.0849 90)
 			(effects
@@
 		(instances
 			(project "1s3p_battery_board"
-				(path "/695f882b-5312-4493-b26d-8f7d6768a9db/7f8fc7f5-7f1e-476b-9e93-5575de1d6778"
-					(reference "R10")
-					(unit 1)
-				)
-			)
-		)
-	)
-	(symbol
-		(lib_id "Connector:TestPoint_Probe")
-		(at 88.9 72.39 0)
-		(mirror y)
-		(unit 1)
-		(exclude_from_sim no)
-		(in_bom no)
-		(on_board yes)
-		(dnp no)
-		(property "Reference" "TP3"
-			(at 85.09 69.5325 0)
-			(effects
-				(font
-					(size 1.27 1.27)
-				)
-				(justify left)
-			)
-		)
-		(property "Value" "GND"
-			(at 85.09 72.0725 0)
-			(effects
-				(font
-					(size 1.27 1.27)
-				)
-				(justify left)
-				(hide yes)
-			)
-		)
-		(property "Footprint" "footprints:TestPoint_Pad_D1.5mm"
-			(at 83.82 72.39 0)
-			(effects
-				(font
-					(size 1.27 1.27)
-				)
-				(hide yes)
-			)
-		)
-		(property "Datasheet" "~"
-			(at 83.82 72.39 0)
-			(effects
-				(font
-					(size 1.27 1.27)
-				)
-				(hide yes)
-			)
-		)
-		(property "Description" "test point (alternative probe-style design)"
-			(at 88.9 72.39 0)
-			(effects
-				(font
-					(size 1.27 1.27)
-				)
-				(hide yes)
-			)
-		)
-		(property "MPN" "NA"
-			(at 88.9 72.39 0)
-			(effects
-				(font
-					(size 1.27 1.27)
-				)
-				(hide yes)
-			)
-		)
-		(property "Active" "Y"
-			(at 88.9 72.39 0)
-			(effects
-				(font
-					(size 1.27 1.27)
-				)
-				(hide yes)
-			)
-		)
-		(property "Basic or Extended Component" ""
-			(at 88.9 72.39 0)
-			(effects
-				(font
-					(size 1.27 1.27)
-				)
-				(hide yes)
-			)
-		)
-		(property "Sim.Device" ""
-			(at 88.9 72.39 0)
-			(effects
-				(font
-					(size 1.27 1.27)
-				)
-				(hide yes)
-			)
-		)
-		(property "Sim.Pins" ""
-			(at 88.9 72.39 0)
-			(effects
-				(font
-					(size 1.27 1.27)
-				)
-				(hide yes)
-			)
-		)
-		(property "Sim.Type" ""
-			(at 88.9 72.39 0)
-			(effects
-				(font
-					(size 1.27 1.27)
-				)
-				(hide yes)
-			)
-		)
-		(pin "1"
-		)
-		(instances
-			(project "1s3p_battery_board"
-				(path "/695f882b-5312-4493-b26d-8f7d6768a9db/7f8fc7f5-7f1e-476b-9e93-5575de1d6778"
-					(reference "TP3")
+				(path "/695f882b-5312-4493-b26d-8f7d6768a9db/64470299-6c65-479c-8ce7-e6a986c7fce1"
+					(reference "R36")
 					(unit 1)
 				)
@@
 		(on_board yes)
 		(dnp no)
-		(property "Reference" "#PWR88"
+		(property "Reference" "#PWR044"
 			(at 88.9 85.09 0)
 			(effects
@@
 		(instances
 			(project "1s3p_battery_board"
-				(path "/695f882b-5312-4493-b26d-8f7d6768a9db/7f8fc7f5-7f1e-476b-9e93-5575de1d6778"
-					(reference "#PWR88")
+				(path "/695f882b-5312-4493-b26d-8f7d6768a9db/64470299-6c65-479c-8ce7-e6a986c7fce1"
+					(reference "#PWR044")
 					(unit 1)
 				)
@@
 		(dnp no)
 		(fields_autoplaced yes)
-		(property "Reference" "#FLG3"
+		(property "Reference" "#FLG04"
 			(at 220.98 40.005 0)
 			(effects
@@
 		(instances
 			(project "1s3p_battery_board"
-				(path "/695f882b-5312-4493-b26d-8f7d6768a9db/7f8fc7f5-7f1e-476b-9e93-5575de1d6778"
-					(reference "#FLG3")
+				(path "/695f882b-5312-4493-b26d-8f7d6768a9db/64470299-6c65-479c-8ce7-e6a986c7fce1"
+					(reference "#FLG04")
 					(unit 1)
 				)
@@
 		(on_board yes)
 		(dnp no)
-		(property "Reference" "C27"
+		(property "Reference" "C38"
 			(at 54.61 48.26 0)
 			(effects
@@
 		(instances
 			(project "1s3p_battery_board"
-				(path "/695f882b-5312-4493-b26d-8f7d6768a9db/7f8fc7f5-7f1e-476b-9e93-5575de1d6778"
-					(reference "C27")
+				(path "/695f882b-5312-4493-b26d-8f7d6768a9db/64470299-6c65-479c-8ce7-e6a986c7fce1"
+					(reference "C38")
 					(unit 1)
 				)
@@
 		(on_board yes)
 		(dnp no)
-		(property "Reference" "C4"
+		(property "Reference" "C39"
 			(at 64.77 48.26 0)
 			(effects
@@
 		(instances
 			(project "1s3p_battery_board"
-				(path "/695f882b-5312-4493-b26d-8f7d6768a9db/7f8fc7f5-7f1e-476b-9e93-5575de1d6778"
-					(reference "C4")
+				(path "/695f882b-5312-4493-b26d-8f7d6768a9db/64470299-6c65-479c-8ce7-e6a986c7fce1"
+					(reference "C39")
 					(unit 1)
 				)
@@
 		(dnp no)
 		(fields_autoplaced yes)
-		(property "Reference" "C6"
+		(property "Reference" "C41"
 			(at 170.18 71.12 0)
 			(effects
@@
 		(instances
 			(project "1s3p_battery_board"
-				(path "/695f882b-5312-4493-b26d-8f7d6768a9db/7f8fc7f5-7f1e-476b-9e93-5575de1d6778"
-					(reference "C6")
+				(path "/695f882b-5312-4493-b26d-8f7d6768a9db/64470299-6c65-479c-8ce7-e6a986c7fce1"
+					(reference "C41")
 					(unit 1)
 				)
@@
 		(on_board yes)
 		(dnp no)
-		(property "Reference" "#PWR89"
+		(property "Reference" "#PWR045"
 			(at 106.68 69.85 0)
 			(effects
@@
 		(instances
 			(project "1s3p_battery_board"
-				(path "/695f882b-5312-4493-b26d-8f7d6768a9db/7f8fc7f5-7f1e-476b-9e93-5575de1d6778"
-					(reference "#PWR89")
+				(path "/695f882b-5312-4493-b26d-8f7d6768a9db/64470299-6c65-479c-8ce7-e6a986c7fce1"
+					(reference "#PWR045")
 					(unit 1)
 				)
@@
 		(dnp no)
 		(fields_autoplaced yes)
-		(property "Reference" "#PWR19"
+		(property "Reference" "#PWR049"
 			(at 180.34 130.81 0)
 			(effects
@@
 		(instances
 			(project "1s3p_battery_board"
-				(path "/695f882b-5312-4493-b26d-8f7d6768a9db/7f8fc7f5-7f1e-476b-9e93-5575de1d6778"
-					(reference "#PWR19")
+				(path "/695f882b-5312-4493-b26d-8f7d6768a9db/64470299-6c65-479c-8ce7-e6a986c7fce1"
+					(reference "#PWR049")
 					(unit 1)
 				)
@@
 		(dnp no)
 		(fields_autoplaced yes)
-		(property "Reference" "C5"
+		(property "Reference" "C40"
 			(at 120.65 48.26 0)
 			(effects
@@
 		(instances
 			(project "1s3p_battery_board"
-				(path "/695f882b-5312-4493-b26d-8f7d6768a9db/7f8fc7f5-7f1e-476b-9e93-5575de1d6778"
-					(reference "C5")
+				(path "/695f882b-5312-4493-b26d-8f7d6768a9db/64470299-6c65-479c-8ce7-e6a986c7fce1"
+					(reference "C40")
 					(unit 1)
 				)

Commit message: Add hierarchical sheet and PCB layout for the core board, including the system bus.
Parts:
- renumbered C38 to C701, C39 to C702, C40 to C703, C41 to C704, C42 to C705, L2 to L701, R35 to R701, R36 to R702, R40 to R703, TP3 to TP701, U5 to U701, U8 to U702
Changed lines of the file:
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@@
 		(on_board yes)
 		(dnp no)
-		(property "Reference" "L2"
+		(property "Reference" "L701"
 			(at 76.2 55.8799 0)
 			(effects
@@
 			(project "1s3p_battery_board"
 				(path "/695f882b-5312-4493-b26d-8f7d6768a9db/64470299-6c65-479c-8ce7-e6a986c7fce1"
-					(reference "L2")
+					(reference "L701")
 					(unit 1)
 				)
@@
 		(on_board yes)
 		(dnp no)
-		(property "Reference" "U5"
+		(property "Reference" "U701"
 			(at 88.9 34.29 0)
 			(effects
@@
 			(project "1s3p_battery_board"
 				(path "/695f882b-5312-4493-b26d-8f7d6768a9db/64470299-6c65-479c-8ce7-e6a986c7fce1"
-					(reference "U5")
+					(reference "U701")
 					(unit 1)
 				)
@@
 		(on_board yes)
 		(dnp no)
-		(property "Reference" "R35"
+		(property "Reference" "R701"
 			(at 102.87 46.99 90)
 			(effects
@@
 			(project "1s3p_battery_board"
 				(path "/695f882b-5312-4493-b26d-8f7d6768a9db/64470299-6c65-479c-8ce7-e6a986c7fce1"
-					(reference "R35")
+					(reference "R701")
 					(unit 1)
 				)
@@
 		(on_board yes)
 		(dnp no)
-		(property "Reference" "U8"
+		(property "Reference" "U702"
 			(at 209.804 110.236 0)
 			(effects
@@
 			(project "1s3p_battery_board"
 				(path "/695f882b-5312-4493-b26d-8f7d6768a9db/64470299-6c65-479c-8ce7-e6a986c7fce1"
-					(reference "U8")
+					(reference "U702")
 					(unit 1)
 				)
@@
 		(on_board yes)
 		(dnp no)
-		(property "Reference" "TP3"
+		(property "Reference" "TP701"
 			(at 64.77 39.0525 0)
 			(effects
@@
 			(project "1s3p_battery_board"
 				(path "/695f882b-5312-4493-b26d-8f7d6768a9db/64470299-6c65-479c-8ce7-e6a986c7fce1"
-					(reference "TP3")
+					(reference "TP701")
 					(unit 1)
 				)
@@
 		(on_board yes)
 		(dnp no)
-		(property "Reference" "#PWR048"
+		(property "Reference" "#PWR0703"
 			(at 173.99 82.55 0)
 			(effects
@@
 			(project "1s3p_battery_board"
 				(path "/695f882b-5312-4493-b26d-8f7d6768a9db/64470299-6c65-479c-8ce7-e6a986c7fce1"
-					(reference "#PWR048")
+					(reference "#PWR0703")
 					(unit 1)
 				)
@@
 		(on_board yes)
 		(dnp no)
-		(property "Reference" "C42"
+		(property "Reference" "C705"
 			(at 195.58 71.12 0)
 			(effects
@@
 			(project "1s3p_battery_board"
 				(path "/695f882b-5312-4493-b26d-8f7d6768a9db/64470299-6c65-479c-8ce7-e6a986c7fce1"
-					(reference "C42")
+					(reference "C705")
 					(unit 1)
 				)
@@
 		(dnp no)
 		(fields_autoplaced yes)
-		(property "Reference" "R40"
+		(property "Reference" "R703"
 			(at 213.36 95.2499 0)
 			(effects
@@
 			(project "1s3p_battery_board"
 				(path "/695f882b-5312-4493-b26d-8f7d6768a9db/64470299-6c65-479c-8ce7-e6a986c7fce1"
-					(reference "R40")
+					(reference "R703")
 					(unit 1)
 				)
@@
 		(on_board yes)
 		(dnp no)
-		(property "Reference" "#PWR051"
+		(property "Reference" "#PWR0705"
 			(at 191.77 82.55 0)
 			(effects
@@
 			(project "1s3p_battery_board"
 				(path "/695f882b-5312-4493-b26d-8f7d6768a9db/64470299-6c65-479c-8ce7-e6a986c7fce1"
-					(reference "#PWR051")
+					(reference "#PWR0705")
 					(unit 1)
 				)
@@
 		(on_board yes)
 		(dnp no)
-		(property "Reference" "R36"
+		(property "Reference" "R702"
 			(at 140.335 45.0849 90)
 			(effects
@@
 			(project "1s3p_battery_board"
 				(path "/695f882b-5312-4493-b26d-8f7d6768a9db/64470299-6c65-479c-8ce7-e6a986c7fce1"
-					(reference "R36")
+					(reference "R702")
 					(unit 1)
 				)
@@
 		(on_board yes)
 		(dnp no)
-		(property "Reference" "#PWR044"
+		(property "Reference" "#PWR0701"
 			(at 88.9 85.09 0)
 			(effects
@@
 			(project "1s3p_battery_board"
 				(path "/695f882b-5312-4493-b26d-8f7d6768a9db/64470299-6c65-479c-8ce7-e6a986c7fce1"
-					(reference "#PWR044")
+					(reference "#PWR0701")
 					(unit 1)
 				)
@@
 		(dnp no)
 		(fields_autoplaced yes)
-		(property "Reference" "#FLG04"
+		(property "Reference" "#FLG0701"
 			(at 220.98 40.005 0)
 			(effects
@@
 			(project "1s3p_battery_board"
 				(path "/695f882b-5312-4493-b26d-8f7d6768a9db/64470299-6c65-479c-8ce7-e6a986c7fce1"
-					(reference "#FLG04")
+					(reference "#FLG0701")
 					(unit 1)
 				)
@@
 		(on_board yes)
 		(dnp no)
-		(property "Reference" "C38"
+		(property "Reference" "C701"
 			(at 54.61 48.26 0)
 			(effects
@@
 			(project "1s3p_battery_board"
 				(path "/695f882b-5312-4493-b26d-8f7d6768a9db/64470299-6c65-479c-8ce7-e6a986c7fce1"
-					(reference "C38")
+					(reference "C701")
 					(unit 1)
 				)
@@
 		(on_board yes)
 		(dnp no)
-		(property "Reference" "C39"
+		(property "Reference" "C702"
 			(at 64.77 48.26 0)
 			(effects
@@
 			(project "1s3p_battery_board"
 				(path "/695f882b-5312-4493-b26d-8f7d6768a9db/64470299-6c65-479c-8ce7-e6a986c7fce1"
-					(reference "C39")
+					(reference "C702")
 					(unit 1)
 				)
@@
 		(dnp no)
 		(fields_autoplaced yes)
-		(property "Reference" "C41"
+		(property "Reference" "C704"
 			(at 170.18 71.12 0)
 			(effects
@@
 			(project "1s3p_battery_board"
 				(path "/695f882b-5312-4493-b26d-8f7d6768a9db/64470299-6c65-479c-8ce7-e6a986c7fce1"
-					(reference "C41")
+					(reference "C704")
 					(unit 1)
 				)
@@
 		(on_board yes)
 		(dnp no)
-		(property "Reference" "#PWR045"
+		(property "Reference" "#PWR0702"
 			(at 106.68 69.85 0)
 			(effects
@@
 			(project "1s3p_battery_board"
 				(path "/695f882b-5312-4493-b26d-8f7d6768a9db/64470299-6c65-479c-8ce7-e6a986c7fce1"
-					(reference "#PWR045")
+					(reference "#PWR0702")
 					(unit 1)
 				)
@@
 		(dnp no)
 		(fields_autoplaced yes)
-		(property "Reference" "#PWR049"
+		(property "Reference" "#PWR0704"
 			(at 180.34 130.81 0)
 			(effects
@@
 			(project "1s3p_battery_board"
 				(path "/695f882b-5312-4493-b26d-8f7d6768a9db/64470299-6c65-479c-8ce7-e6a986c7fce1"
-					(reference "#PWR049")
+					(reference "#PWR0704")
 					(unit 1)
 				)
@@
 		(dnp no)
 		(fields_autoplaced yes)
-		(property "Reference" "C40"
+		(property "Reference" "C703"
 			(at 120.65 48.26 0)
 			(effects
@@
 			(project "1s3p_battery_board"
 				(path "/695f882b-5312-4493-b26d-8f7d6768a9db/64470299-6c65-479c-8ce7-e6a986c7fce1"
-					(reference "C40")
+					(reference "C703")
 					(unit 1)
 				)
