File: electrical/pcb_design/1s3p_battery_board/single_solar_accumulator.kicad_sch (KiCad schematic)
At the start: 7 parts, among them U11 SPV1040TTR, U13 LM66100DCK

Commit message: Add hierarchical sheet and PCB layout for the core board, including the system bus.
Parts:
- renumbered L3 to L1101, R42 to R1101, R44 to R1102, R43 to R1103, RV1 to RV1101, U13 to U1101, U11 to U1102
