File: electrical/modules/can_bus/can_bus.kicad_sch (KiCad schematic)
At the start: 8 parts, among them U101 TCAN330DR

Commit message: Checkpoint work on building core board module.
Parts:
- renumbered C101 to C501, C102 to C502, C103 to C503, JP101 to JP501, JP102 to JP502, R101 to R501, R102 to R502, U101 to U501
Changed lines of the file:
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@@
 		(on_board yes)
 		(dnp no)
-		(property "Reference" "C103"
+		(property "Reference" "C503"
 			(at 173.228 77.978 0)
 			(effects
@@
 		)
 		(instances
-			(project "1s3p_battery_board"
-				(path "/695f882b-5312-4493-b26d-8f7d6768a9db/e0e5088b-2fa2-4f34-adc6-d0f708744404/d470ef27-6c0f-4ffa-83b6-2c4b3c9c5ff3"
+			(project "core_board"
+				(path "/695f882b-5312-4493-b26d-8f7d6768a9db/d470ef27-6c0f-4ffa-83b6-2c4b3c9c5ff3"
 					(reference "C503")
 					(unit 1)
@@
 		(on_board yes)
 		(dnp no)
-		(property "Reference" "U101"
+		(property "Reference" "U501"
 			(at 99.568 64.262 0)
 			(effects
@@
 		)
 		(instances
-			(project "1s3p_battery_board"
-				(path "/695f882b-5312-4493-b26d-8f7d6768a9db/e0e5088b-2fa2-4f34-adc6-d0f708744404/d470ef27-6c0f-4ffa-83b6-2c4b3c9c5ff3"
+			(project "core_board"
+				(path "/695f882b-5312-4493-b26d-8f7d6768a9db/d470ef27-6c0f-4ffa-83b6-2c4b3c9c5ff3"
 					(reference "U501")
 					(unit 1)
@@
 		(on_board yes)
 		(dnp no)
-		(property "Reference" "R102"
+		(property "Reference" "R502"
 			(at 185.928 71.882 90)
 			(effects
@@
 		)
 		(instances
-			(project "1s3p_battery_board"
-				(path "/695f882b-5312-4493-b26d-8f7d6768a9db/e0e5088b-2fa2-4f34-adc6-d0f708744404/d470ef27-6c0f-4ffa-83b6-2c4b3c9c5ff3"
+			(project "core_board"
+				(path "/695f882b-5312-4493-b26d-8f7d6768a9db/d470ef27-6c0f-4ffa-83b6-2c4b3c9c5ff3"
 					(reference "R502")
 					(unit 1)
@@
 		(on_board yes)
 		(dnp no)
-		(property "Reference" "#PWR0102"
+		(property "Reference" "#PWR0502"
 			(at 58.42 52.07 0)
 			(effects
@@
 		)
 		(instances
-			(project "1s3p_battery_board"
-				(path "/695f882b-5312-4493-b26d-8f7d6768a9db/e0e5088b-2fa2-4f34-adc6-d0f708744404/d470ef27-6c0f-4ffa-83b6-2c4b3c9c5ff3"
+			(project "core_board"
+				(path "/695f882b-5312-4493-b26d-8f7d6768a9db/d470ef27-6c0f-4ffa-83b6-2c4b3c9c5ff3"
 					(reference "#PWR0502")
 					(unit 1)
@@
 		(on_board yes)
 		(dnp no)
-		(property "Reference" "JP101"
+		(property "Reference" "JP501"
 			(at 144.78 72.39 0)
 			(effects
@@
 		)
 		(instances
-			(project "1s3p_battery_board"
-				(path "/695f882b-5312-4493-b26d-8f7d6768a9db/e0e5088b-2fa2-4f34-adc6-d0f708744404/d470ef27-6c0f-4ffa-83b6-2c4b3c9c5ff3"
+			(project "core_board"
+				(path "/695f882b-5312-4493-b26d-8f7d6768a9db/d470ef27-6c0f-4ffa-83b6-2c4b3c9c5ff3"
 					(reference "JP501")
 					(unit 1)
@@
 		(on_board yes)
 		(dnp no)
-		(property "Reference" "#PWR0101"
+		(property "Reference" "#PWR0501"
 			(at 55.88 71.12 0)
 			(effects
@@
 		)
 		(instances
-			(project "1s3p_battery_board"
-				(path "/695f882b-5312-4493-b26d-8f7d6768a9db/e0e5088b-2fa2-4f34-adc6-d0f708744404/d470ef27-6c0f-4ffa-83b6-2c4b3c9c5ff3"
+			(project "core_board"
+				(path "/695f882b-5312-4493-b26d-8f7d6768a9db/d470ef27-6c0f-4ffa-83b6-2c4b3c9c5ff3"
 					(reference "#PWR0501")
 					(unit 1)
@@
 		(on_board yes)
 		(dnp no)
-		(property "Reference" "#PWR0103"
+		(property "Reference" "#PWR0503"
 			(at 179.07 88.9 0)
 			(effects
@@
 		)
 		(instances
-			(project "1s3p_battery_board"
-				(path "/695f882b-5312-4493-b26d-8f7d6768a9db/e0e5088b-2fa2-4f34-adc6-d0f708744404/d470ef27-6c0f-4ffa-83b6-2c4b3c9c5ff3"
+			(project "core_board"
+				(path "/695f882b-5312-4493-b26d-8f7d6768a9db/d470ef27-6c0f-4ffa-83b6-2c4b3c9c5ff3"
 					(reference "#PWR0503")
 					(unit 1)
@@
 		(on_board yes)
 		(dnp no)
-		(property "Reference" "JP102"
+		(property "Reference" "JP502"
 			(at 212.09 72.39 0)
 			(effects
@@
 		)
 		(instances
-			(project "1s3p_battery_board"
-				(path "/695f882b-5312-4493-b26d-8f7d6768a9db/e0e5088b-2fa2-4f34-adc6-d0f708744404/d470ef27-6c0f-4ffa-83b6-2c4b3c9c5ff3"
+			(project "core_board"
+				(path "/695f882b-5312-4493-b26d-8f7d6768a9db/d470ef27-6c0f-4ffa-83b6-2c4b3c9c5ff3"
 					(reference "JP502")
 					(unit 1)
@@
 		(dnp no)
 		(fields_autoplaced yes)
-		(property "Reference" "C102"
+		(property "Reference" "C502"
 			(at 64.77 59.69 0)
 			(effects
@@
 		)
 		(instances
-			(project "1s3p_battery_board"
-				(path "/695f882b-5312-4493-b26d-8f7d6768a9db/e0e5088b-2fa2-4f34-adc6-d0f708744404/d470ef27-6c0f-4ffa-83b6-2c4b3c9c5ff3"
+			(project "core_board"
+				(path "/695f882b-5312-4493-b26d-8f7d6768a9db/d470ef27-6c0f-4ffa-83b6-2c4b3c9c5ff3"
 					(reference "C502")
 					(unit 1)
@@
 		(on_board yes)
 		(dnp no)
-		(property "Reference" "R101"
+		(property "Reference" "R501"
 			(at 172.466 71.882 90)
 			(effects
@@
 		)
 		(instances
-			(project "1s3p_battery_board"
-				(path "/695f882b-5312-4493-b26d-8f7d6768a9db/e0e5088b-2fa2-4f34-adc6-d0f708744404/d470ef27-6c0f-4ffa-83b6-2c4b3c9c5ff3"
+			(project "core_board"
+				(path "/695f882b-5312-4493-b26d-8f7d6768a9db/d470ef27-6c0f-4ffa-83b6-2c4b3c9c5ff3"
 					(reference "R501")
 					(unit 1)
@@
 		(dnp no)
 		(fields_autoplaced yes)
-		(property "Reference" "C101"
+		(property "Reference" "C501"
 			(at 53.34 59.69 0)
 			(effects
@@
 		)
 		(instances
-			(project "1s3p_battery_board"
-				(path "/695f882b-5312-4493-b26d-8f7d6768a9db/e0e5088b-2fa2-4f34-adc6-d0f708744404/d470ef27-6c0f-4ffa-83b6-2c4b3c9c5ff3"
+			(project "core_board"
+				(path "/695f882b-5312-4493-b26d-8f7d6768a9db/d470ef27-6c0f-4ffa-83b6-2c4b3c9c5ff3"
 					(reference "C501")
 					(unit 1)

Commit message: Checkpoint layout work on 1s3p battery board. This change includes many updates to modules, including design changes to avoid mechanical conflicts with battery placements. Some of these changes are noise due to limitations in KiCad 9.
Parts:
- renumbered C501 to C1101, C502 to C1102, C503 to C1103, JP501 to JP1101, JP502 to JP1102, R501 to R1101, R502 to R1102, U501 to U1101
Changed lines of the file:
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@@
 		(on_board yes)
 		(dnp no)
-		(property "Reference" "C503"
+		(property "Reference" "C1103"
 			(at 173.228 77.978 0)
 			(effects
@@
 		)
 		(instances
-			(project "core_board"
-				(path "/695f882b-5312-4493-b26d-8f7d6768a9db/d470ef27-6c0f-4ffa-83b6-2c4b3c9c5ff3"
-					(reference "C503")
+			(project "1s3p_battery_board"
+				(path "/695f882b-5312-4493-b26d-8f7d6768a9db/e0e5088b-2fa2-4f34-adc6-d0f708744404/d470ef27-6c0f-4ffa-83b6-2c4b3c9c5ff3"
+					(reference "C1103")
 					(unit 1)
 				)
@@
 		(on_board yes)
 		(dnp no)
-		(property "Reference" "U501"
+		(property "Reference" "U1101"
 			(at 99.568 64.262 0)
 			(effects
@@
 		)
 		(instances
-			(project "core_board"
-				(path "/695f882b-5312-4493-b26d-8f7d6768a9db/d470ef27-6c0f-4ffa-83b6-2c4b3c9c5ff3"
-					(reference "U501")
+			(project "1s3p_battery_board"
+				(path "/695f882b-5312-4493-b26d-8f7d6768a9db/e0e5088b-2fa2-4f34-adc6-d0f708744404/d470ef27-6c0f-4ffa-83b6-2c4b3c9c5ff3"
+					(reference "U1101")
 					(unit 1)
 				)
@@
 		(on_board yes)
 		(dnp no)
-		(property "Reference" "R502"
+		(property "Reference" "R1102"
 			(at 185.928 71.882 90)
 			(effects
@@
 		)
 		(instances
-			(project "core_board"
-				(path "/695f882b-5312-4493-b26d-8f7d6768a9db/d470ef27-6c0f-4ffa-83b6-2c4b3c9c5ff3"
-					(reference "R502")
+			(project "1s3p_battery_board"
+				(path "/695f882b-5312-4493-b26d-8f7d6768a9db/e0e5088b-2fa2-4f34-adc6-d0f708744404/d470ef27-6c0f-4ffa-83b6-2c4b3c9c5ff3"
+					(reference "R1102")
 					(unit 1)
 				)
@@
 		(on_board yes)
 		(dnp no)
-		(property "Reference" "#PWR0502"
+		(property "Reference" "#PWR01102"
 			(at 58.42 52.07 0)
 			(effects
@@
 		)
 		(instances
-			(project "core_board"
-				(path "/695f882b-5312-4493-b26d-8f7d6768a9db/d470ef27-6c0f-4ffa-83b6-2c4b3c9c5ff3"
-					(reference "#PWR0502")
+			(project "1s3p_battery_board"
+				(path "/695f882b-5312-4493-b26d-8f7d6768a9db/e0e5088b-2fa2-4f34-adc6-d0f708744404/d470ef27-6c0f-4ffa-83b6-2c4b3c9c5ff3"
+					(reference "#PWR01102")
 					(unit 1)
 				)
@@
 		(on_board yes)
 		(dnp no)
-		(property "Reference" "JP501"
+		(property "Reference" "JP1101"
 			(at 144.78 72.39 0)
 			(effects
@@
 		)
 		(instances
-			(project "core_board"
-				(path "/695f882b-5312-4493-b26d-8f7d6768a9db/d470ef27-6c0f-4ffa-83b6-2c4b3c9c5ff3"
-					(reference "JP501")
+			(project "1s3p_battery_board"
+				(path "/695f882b-5312-4493-b26d-8f7d6768a9db/e0e5088b-2fa2-4f34-adc6-d0f708744404/d470ef27-6c0f-4ffa-83b6-2c4b3c9c5ff3"
+					(reference "JP1101")
 					(unit 1)
 				)
@@
 		(on_board yes)
 		(dnp no)
-		(property "Reference" "#PWR0501"
+		(property "Reference" "#PWR01101"
 			(at 55.88 71.12 0)
 			(effects
@@
 		)
 		(instances
-			(project "core_board"
-				(path "/695f882b-5312-4493-b26d-8f7d6768a9db/d470ef27-6c0f-4ffa-83b6-2c4b3c9c5ff3"
-					(reference "#PWR0501")
+			(project "1s3p_battery_board"
+				(path "/695f882b-5312-4493-b26d-8f7d6768a9db/e0e5088b-2fa2-4f34-adc6-d0f708744404/d470ef27-6c0f-4ffa-83b6-2c4b3c9c5ff3"
+					(reference "#PWR01101")
 					(unit 1)
 				)
@@
 		(on_board yes)
 		(dnp no)
-		(property "Reference" "#PWR0503"
+		(property "Reference" "#PWR01103"
 			(at 179.07 88.9 0)
 			(effects
@@
 		)
 		(instances
-			(project "core_board"
-				(path "/695f882b-5312-4493-b26d-8f7d6768a9db/d470ef27-6c0f-4ffa-83b6-2c4b3c9c5ff3"
-					(reference "#PWR0503")
+			(project "1s3p_battery_board"
+				(path "/695f882b-5312-4493-b26d-8f7d6768a9db/e0e5088b-2fa2-4f34-adc6-d0f708744404/d470ef27-6c0f-4ffa-83b6-2c4b3c9c5ff3"
+					(reference "#PWR01103")
 					(unit 1)
 				)
@@
 		(on_board yes)
 		(dnp no)
-		(property "Reference" "JP502"
+		(property "Reference" "JP1102"
 			(at 212.09 72.39 0)
 			(effects
@@
 		)
 		(instances
-			(project "core_board"
-				(path "/695f882b-5312-4493-b26d-8f7d6768a9db/d470ef27-6c0f-4ffa-83b6-2c4b3c9c5ff3"
-					(reference "JP502")
+			(project "1s3p_battery_board"
+				(path "/695f882b-5312-4493-b26d-8f7d6768a9db/e0e5088b-2fa2-4f34-adc6-d0f708744404/d470ef27-6c0f-4ffa-83b6-2c4b3c9c5ff3"
+					(reference "JP1102")
 					(unit 1)
 				)
@@
 		(dnp no)
 		(fields_autoplaced yes)
-		(property "Reference" "C502"
+		(property "Reference" "C1102"
 			(at 64.77 59.69 0)
 			(effects
@@
 		)
 		(instances
-			(project "core_board"
-				(path "/695f882b-5312-4493-b26d-8f7d6768a9db/d470ef27-6c0f-4ffa-83b6-2c4b3c9c5ff3"
-					(reference "C502")
+			(project "1s3p_battery_board"
+				(path "/695f882b-5312-4493-b26d-8f7d6768a9db/e0e5088b-2fa2-4f34-adc6-d0f708744404/d470ef27-6c0f-4ffa-83b6-2c4b3c9c5ff3"
+					(reference "C1102")
 					(unit 1)
 				)
@@
 		(on_board yes)
 		(dnp no)
-		(property "Reference" "R501"
+		(property "Reference" "R1101"
 			(at 172.466 71.882 90)
 			(effects
@@
 		)
 		(instances
-			(project "core_board"
-				(path "/695f882b-5312-4493-b26d-8f7d6768a9db/d470ef27-6c0f-4ffa-83b6-2c4b3c9c5ff3"
-					(reference "R501")
+			(project "1s3p_battery_board"
+				(path "/695f882b-5312-4493-b26d-8f7d6768a9db/e0e5088b-2fa2-4f34-adc6-d0f708744404/d470ef27-6c0f-4ffa-83b6-2c4b3c9c5ff3"
+					(reference "R1101")
 					(unit 1)
 				)
@@
 		(dnp no)
 		(fields_autoplaced yes)
-		(property "Reference" "C501"
+		(property "Reference" "C1101"
 			(at 53.34 59.69 0)
 			(effects
@@
 		)
 		(instances
-			(project "core_board"
-				(path "/695f882b-5312-4493-b26d-8f7d6768a9db/d470ef27-6c0f-4ffa-83b6-2c4b3c9c5ff3"
-					(reference "C501")
-					(unit 1)
-				)
+			(project "1s3p_battery_board"
+				(path "/695f882b-5312-4493-b26d-8f7d6768a9db/e0e5088b-2fa2-4f34-adc6-d0f708744404/d470ef27-6c0f-4ffa-83b6-2c4b3c9c5ff3"
+					(reference "C1101")
+					(unit 1)
+				)
