File: electronics/common/blocks/pcb_with_bus/pcb_with_bus.kicad_sch (KiCad schematic)
At the start: 5 parts, among them J201 QTH-030-07-L-D-A, J202 QSH-030-01-L-D-A

Commit message: Structure the PCB with system bus headers design block so that it passes ERC and DRC without issues, has proper page size, includes version and name information, etc.
Parts:
- PCB202: renamed from PCB201; value ~ -> (none)
- renumbered D201 to D202, J201 to J203, J202 to J204, R201 to R202
