File: electronics/projects/blocks/power_measurement/power_measurement.kicad_pcb (KiCad board)
At the start: 4 copper layers, 4 parts, among them U401 PAC1934T-I/JQ

Commit message: Create project to manage power measurement design block.
Connections:
- net /3V3 renamed /power_measurement/3V3
- net /BOARD_LOAD_+ renamed /power_measurement/BOARD_LOAD_+
- net /I2C_SCL renamed /power_measurement/I2C_SCL
- net /I2C_SDA renamed /power_measurement/I2C_SDA
- net /SENSE_2_+ renamed /power_measurement/SENSE_2_+
- net /SENSE_2_- renamed /power_measurement/SENSE_2_-
- net /SENSE_3_+ renamed /power_measurement/SENSE_3_+
- net /SENSE_3_- renamed /power_measurement/SENSE_3_-
- net /SENSE_4_+ renamed /power_measurement/SENSE_4_+
- net /SENSE_4_- renamed /power_measurement/SENSE_4_-
