File: electronics/common/library.kicad_blocks/voltage_regulation.kicad_block/voltage_regulation.kicad_pcb (KiCad board)
At the start: 4 copper layers, 7 parts, among them U301 TPS63900

Commit message: Try another approach with design blocks. This approach annotates all components in the design block based around page number x 100, where the primary page for each design block starts at page 1.
Parts:
- renumbered C301 to C101, C302 to C102, C303 to C103, L301 to L101, R301 to R101, R302 to R102, U301 to U101
Routing:
- net /Voltage Regulation/BOARD_LOAD_+: track 5.62 -> 0.00 mm
Changed lines of the file:
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@@
 		(descr "Capacitor SMD 0603 (1608 Metric), square (rectangular) end terminal, IPC_7351 nominal, (Body size source: IPC-SM-782 page 76, https://www.pcb-3d.com/wordpress/wp-content/uploads/ipc-sm-782a_amendment_1_and_2.pdf), generated with kicad-footprint-generator")
 		(tags "capacitor")
-		(property "Reference" "C301"
+		(property "Reference" "C101"
 			(at 0 1.43 90)
 			(layer "B.SilkS")
@@
 		(descr "Capacitor SMD 0603 (1608 Metric), square (rectangular) end terminal, IPC_7351 nominal, (Body size source: IPC-SM-782 page 76, https://www.pcb-3d.com/wordpress/wp-content/uploads/ipc-sm-782a_amendment_1_and_2.pdf), generated with kicad-footprint-generator")
 		(tags "capacitor")
-		(property "Reference" "C302"
+		(property "Reference" "C102"
 			(at 0 1.43 90)
 			(layer "B.SilkS")
@@
 		(descr "WSON, 10 Pin (http://www.ti.com/lit/gpn/tps63030#page=24), generated with kicad-footprint-generator ipc_noLead_generator.py")
 		(tags "WSON NoLead")
-		(property "Reference" "U301"
+		(property "Reference" "U101"
 			(at 0 2.2 90)
 			(layer "B.Fab")
@@
 			(layers "B.Cu" "B.Mask" "B.Paste")
 			(roundrect_rratio 0.25)
-			(net "Net-(U301-CFG1)")
+			(net "Net-(U101-CFG1)")
 			(pinfunction "CFG1_3")
 			(pintype "input")
@@
 			(layers "B.Cu" "B.Mask" "B.Paste")
 			(roundrect_rratio 0.25)
-			(net "Net-(U301-LX2)")
+			(net "Net-(U101-LX2)")
 			(pinfunction "LX2_7")
 			(pintype "input")
@@
 			(layers "B.Cu" "B.Mask" "B.Paste")
 			(roundrect_rratio 0.25)
-			(net "Net-(U301-LX1)")
+			(net "Net-(U101-LX1)")
 			(pinfunction "LX1_9")
 			(pintype "input")
@@
 		(descr "Inductor SMD 1008 (2520 Metric), square (rectangular) end terminal, IPC-7351 nominal, (Body size source: https://ecsxtal.com/store/pdf/ECS-MPI2520-SMD-POWER-INDUCTOR.pdf), generated with kicad-footprint-generator")
 		(tags "inductor")
-		(property "Reference" "L301"
+		(property "Reference" "L101"
 			(at 0 2.05 0)
 			(layer "B.SilkS")
@@
 			(layers "B.Cu" "B.Mask" "B.Paste")
 			(roundrect_rratio 0.2)
-			(net "Net-(U301-LX2)")
+			(net "Net-(U101-LX2)")
 			(pintype "passive")
 		)
@@
 			(layers "B.Cu" "B.Mask" "B.Paste")
 			(roundrect_rratio 0.2)
-			(net "Net-(U301-LX1)")
+			(net "Net-(U101-LX1)")
 			(pintype "passive")
 		)
@@
 		(descr "Resistor SMD 0805 (2012 Metric), square (rectangular) end terminal, IPC-7351 nominal, (Body size source: IPC-SM-782 page 72, https://www.pcb-3d.com/wordpress/wp-content/uploads/ipc-sm-782a_amendment_1_and_2.pdf), generated with kicad-footprint-generator")
 		(tags "resistor")
-		(property "Reference" "R302"
+		(property "Reference" "R102"
 			(at 0 1.65 0)
 			(layer "B.SilkS")
@@
 		(descr "Capacitor SMD 0603 (1608 Metric), square (rectangular) end terminal, IPC_7351 nominal, (Body size source: IPC-SM-782 page 76, https://www.pcb-3d.com/wordpress/wp-content/uploads/ipc-sm-782a_amendment_1_and_2.pdf), generated with kicad-footprint-generator")
 		(tags "capacitor")
-		(property "Reference" "C303"
+		(property "Reference" "C103"
 			(at 0 1.43 90)
 			(layer "B.SilkS")
@@
 		(descr "Resistor SMD 0402 (1005 Metric), square (rectangular) end terminal, IPC_7351 nominal, (Body size source: IPC-SM-782 page 72, https://www.pcb-3d.com/wordpress/wp-content/uploads/ipc-sm-782a_amendment_1_and_2.pdf), generated with kicad-footprint-generator")
 		(tags "resistor")
-		(property "Reference" "R301"
+		(property "Reference" "R101"
 			(at 0 1.17 0)
 			(layer "B.SilkS")
@@
 			(layers "B.Cu" "B.Mask" "B.Paste")
 			(roundrect_rratio 0.25)
-			(net "Net-(U301-CFG1)")
+			(net "Net-(U101-CFG1)")
 			(pintype "passive")
 		)
@@
 		(net "GND")
 	)
-	(segment
-		(start 144.15 94.975)
-		(end 144.16 94.965)
-		(width 0.3)
-		(layer "B.Cu")
-		(net "Net-(U301-CFG1)")
-	)
-	(segment
-		(start 144.15 96.1325)
-		(end 144.15 94.975)
-		(width 0.3)
-		(layer "B.Cu")
-		(net "Net-(U301-CFG1)")
-	)
-	(segment
-		(start 147.9875 98.495)
-		(end 147.9875 99.5125)
-		(width 0.3)
-		(layer "B.Cu")
-		(net "/Voltage Regulation/BOARD_LOAD_+")
-	)
-	(segment
-		(start 147.9875 99.5125)
-		(end 148.77 100.295)
-		(width 0.3)
-		(layer "B.Cu")
-		(net "/Voltage Regulation/BOARD_LOAD_+")
-	)
-	(segment
-		(start 148.77 100.295)
-		(end 152.27 100.295)
-		(width 0.3)
-		(layer "B.Cu")
-		(net "/Voltage Regulation/BOARD_LOAD_+")
-	)
 	(via
 		(at 151.25 98.495)
@@
 		(net "/Voltage Regulation/3V3")
 	)
+	(segment
+		(start 144.15 94.975)
+		(end 144.16 94.965)
+		(width 0.3)
+		(layer "B.Cu")
+		(net "Net-(U101-CFG1)")
+	)
+	(segment
+		(start 144.15 96.1325)
+		(end 144.15 94.975)
+		(width 0.3)
+		(layer "B.Cu")
+		(net "Net-(U101-CFG1)")
+	)
 	(zone
-		(net "Net-(U301-LX2)")
+		(net "Net-(U101-LX2)")
 		(layer "B.Cu")
 		(hatch edge 0.5)
@@
 	)
 	(zone
-		(net "Net-(U301-LX1)")
+		(net "Net-(U101-LX1)")
 		(layer "B.Cu")
 		(hatch edge 0.5)

Commit message: Update voltage regulation design block to tune copper fills to give better connection for power rails and switching inductor.
Routing:
- net GND: track 1.76 -> 1.70 mm, vias 23 -> 26
