File: electronics/projects/blocks/voltage_regulation/voltage_regulation.kicad_sch (KiCad schematic)
At the start: 7 parts, among them U301 TPS63900

Commit message: Try another approach with design blocks. This approach annotates all components in the design block based around page number x 100, where the primary page for each design block starts at page 1.
Parts:
- renumbered C301 to C101, C302 to C102, C303 to C103, L301 to L101, R301 to R101, R302 to R102, U301 to U101
Changed lines of the file:
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@@
 		(in_pos_files yes)
 		(dnp no)
-		(property "Reference" "L301"
+		(property "Reference" "L101"
 			(at 83.82 62.2299 0)
 			(show_name no)
@@
 		)
 		(instances
-			(project "voltage_regulation"
-				(path "/5f5e286b-eaca-457b-b591-57ed7664ba4e"
-					(reference "L301")
-					(unit 1)
-				)
-			)
 			(project "core_board"
 				(path "/695f882b-5312-4493-b26d-8f7d6768a9db/64470299-6c65-479c-8ce7-e6a986c7fce1"
@@
 			(project "voltage_regulation"
 				(path "/c5d96ab9-5a29-4a9c-8454-97d11b1b2425/2e3bd425-bc2a-4575-ae86-3cfba4ed8b03"
-					(reference "L301")
+					(reference "L101")
 					(unit 1)
 				)
@@
 		(in_pos_files yes)
 		(dnp no)
-		(property "Reference" "U301"
+		(property "Reference" "U101"
 			(at 96.52 40.64 0)
 			(show_name no)
@@
 		)
 		(instances
-			(project "voltage_regulation"
-				(path "/5f5e286b-eaca-457b-b591-57ed7664ba4e"
-					(reference "U301")
-					(unit 1)
-				)
-			)
 			(project "core_board"
 				(path "/695f882b-5312-4493-b26d-8f7d6768a9db/64470299-6c65-479c-8ce7-e6a986c7fce1"
@@
 			(project "voltage_regulation"
 				(path "/c5d96ab9-5a29-4a9c-8454-97d11b1b2425/2e3bd425-bc2a-4575-ae86-3cfba4ed8b03"
-					(reference "U301")
+					(reference "U101")
 					(unit 1)
 				)
@@
 		(in_pos_files yes)
 		(dnp no)
-		(property "Reference" "R301"
+		(property "Reference" "R101"
 			(at 110.49 53.34 90)
 			(show_name no)
@@
 		)
 		(instances
-			(project "voltage_regulation"
-				(path "/5f5e286b-eaca-457b-b591-57ed7664ba4e"
-					(reference "R301")
-					(unit 1)
-				)
-			)
 			(project "core_board"
 				(path "/695f882b-5312-4493-b26d-8f7d6768a9db/64470299-6c65-479c-8ce7-e6a986c7fce1"
@@
 			(project "voltage_regulation"
 				(path "/c5d96ab9-5a29-4a9c-8454-97d11b1b2425/2e3bd425-bc2a-4575-ae86-3cfba4ed8b03"
-					(reference "R301")
+					(reference "R101")
 					(unit 1)
 				)
@@
 		(in_pos_files yes)
 		(dnp no)
-		(property "Reference" "R302"
+		(property "Reference" "R102"
 			(at 147.955 51.4349 90)
 			(show_name no)
@@
 		)
 		(instances
-			(project "voltage_regulation"
-				(path "/5f5e286b-eaca-457b-b591-57ed7664ba4e"
-					(reference "R302")
-					(unit 1)
-				)
-			)
 			(project "core_board"
 				(path "/695f882b-5312-4493-b26d-8f7d6768a9db/64470299-6c65-479c-8ce7-e6a986c7fce1"
@@
 			(project "voltage_regulation"
 				(path "/c5d96ab9-5a29-4a9c-8454-97d11b1b2425/2e3bd425-bc2a-4575-ae86-3cfba4ed8b03"
-					(reference "R302")
+					(reference "R102")
 					(unit 1)
 				)
@@
 		(in_pos_files yes)
 		(dnp no)
-		(property "Reference" "#PWR0301"
+		(property "Reference" "#PWR0101"
 			(at 96.52 91.44 0)
 			(hide yes)
@@
 		)
 		(instances
-			(project "voltage_regulation"
-				(path "/5f5e286b-eaca-457b-b591-57ed7664ba4e"
-					(reference "#PWR0301")
-					(unit 1)
-				)
-			)
 			(project "core_board"
 				(path "/695f882b-5312-4493-b26d-8f7d6768a9db/64470299-6c65-479c-8ce7-e6a986c7fce1"
@@
 			(project "voltage_regulation"
 				(path "/c5d96ab9-5a29-4a9c-8454-97d11b1b2425/2e3bd425-bc2a-4575-ae86-3cfba4ed8b03"
-					(reference "#PWR0301")
+					(reference "#PWR0101")
 					(unit 1)
 				)
@@
 		(dnp no)
 		(fields_autoplaced yes)
-		(property "Reference" "#FLG0301"
+		(property "Reference" "#FLG0101"
 			(at 228.6 46.355 0)
 			(hide yes)
@@
 		)
 		(instances
-			(project "voltage_regulation"
-				(path "/5f5e286b-eaca-457b-b591-57ed7664ba4e"
-					(reference "#FLG0301")
-					(unit 1)
-				)
-			)
 			(project "core_board"
 				(path "/695f882b-5312-4493-b26d-8f7d6768a9db/64470299-6c65-479c-8ce7-e6a986c7fce1"
@@
 			(project "voltage_regulation"
 				(path "/c5d96ab9-5a29-4a9c-8454-97d11b1b2425/2e3bd425-bc2a-4575-ae86-3cfba4ed8b03"
-					(reference "#FLG0301")
+					(reference "#FLG0101")
 					(unit 1)
 				)
@@
 		(in_pos_files yes)
 		(dnp no)
-		(property "Reference" "C301"
+		(property "Reference" "C101"
 			(at 62.23 54.61 0)
 			(show_name no)
@@
 		)
 		(instances
-			(project "voltage_regulation"
-				(path "/5f5e286b-eaca-457b-b591-57ed7664ba4e"
-					(reference "C301")
-					(unit 1)
-				)
-			)
 			(project "core_board"
 				(path "/695f882b-5312-4493-b26d-8f7d6768a9db/64470299-6c65-479c-8ce7-e6a986c7fce1"
@@
 			(project "voltage_regulation"
 				(path "/c5d96ab9-5a29-4a9c-8454-97d11b1b2425/2e3bd425-bc2a-4575-ae86-3cfba4ed8b03"
-					(reference "C301")
+					(reference "C101")
 					(unit 1)
 				)
@@
 		(in_pos_files yes)
 		(dnp no)
-		(property "Reference" "C302"
+		(property "Reference" "C102"
 			(at 72.39 54.61 0)
 			(show_name no)
@@
 		)
 		(instances
-			(project "voltage_regulation"
-				(path "/5f5e286b-eaca-457b-b591-57ed7664ba4e"
-					(reference "C302")
-					(unit 1)
-				)
-			)
 			(project "core_board"
 				(path "/695f882b-5312-4493-b26d-8f7d6768a9db/64470299-6c65-479c-8ce7-e6a986c7fce1"
@@
 			(project "voltage_regulation"
 				(path "/c5d96ab9-5a29-4a9c-8454-97d11b1b2425/2e3bd425-bc2a-4575-ae86-3cfba4ed8b03"
-					(reference "C302")
+					(reference "C102")
 					(unit 1)
 				)
@@
 		(in_pos_files yes)
 		(dnp no)
-		(property "Reference" "#PWR0302"
+		(property "Reference" "#PWR0102"
 			(at 114.3 76.2 0)
 			(hide yes)
@@
 		)
 		(instances
-			(project "voltage_regulation"
-				(path "/5f5e286b-eaca-457b-b591-57ed7664ba4e"
-					(reference "#PWR0302")
-					(unit 1)
-				)
-			)
 			(project "core_board"
 				(path "/695f882b-5312-4493-b26d-8f7d6768a9db/64470299-6c65-479c-8ce7-e6a986c7fce1"
@@
 			(project "voltage_regulation"
 				(path "/c5d96ab9-5a29-4a9c-8454-97d11b1b2425/2e3bd425-bc2a-4575-ae86-3cfba4ed8b03"
-					(reference "#PWR0302")
+					(reference "#PWR0102")
 					(unit 1)
 				)
@@
 		(dnp no)
 		(fields_autoplaced yes)
-		(property "Reference" "C303"
+		(property "Reference" "C103"
 			(at 128.27 54.61 0)
 			(show_name no)
@@
 		)
 		(instances
-			(project "voltage_regulation"
-				(path "/5f5e286b-eaca-457b-b591-57ed7664ba4e"
-					(reference "C303")
-					(unit 1)
-				)
-			)
 			(project "core_board"
 				(path "/695f882b-5312-4493-b26d-8f7d6768a9db/64470299-6c65-479c-8ce7-e6a986c7fce1"
@@
 			(project "voltage_regulation"
 				(path "/c5d96ab9-5a29-4a9c-8454-97d11b1b2425/2e3bd425-bc2a-4575-ae86-3cfba4ed8b03"
-					(reference "C303")
-					(unit 1)
-				)
+					(reference "C103")
+					(unit 1)
+				)

Commit message: Tweak schematic to make the board load pos signal more obviously an output and to better document that GND is driven elsewhere.
Changed lines of the file:
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@@
 	(wire
 		(pts
-			(xy 140.97 45.72) (xy 140.97 48.26)
+			(xy 140.97 63.5) (xy 140.97 48.26)
 		)
 		(stroke
@@
 	(wire
 		(pts
-			(xy 138.43 45.72) (xy 140.97 45.72)
+			(xy 231.14 63.5) (xy 140.97 63.5)
 		)
 		(stroke
@@
 	(hierarchical_label "BOARD_LOAD_+"
 		(shape output)
-		(at 138.43 45.72 180)
+		(at 231.14 63.5 0)
 		(effects
 			(font
 				(size 1.27 1.27)
 			)
-			(justify right)
-		)
-	)
+			(justify left)
+		)
+	)
