File: electronics/projects/blocks/core_board/voltage_regulation.kicad_sch (KiCad schematic)
At the start: 7 parts, among them U501 TPS63900

Commit message: Update all sheets in core board project. Still looking for processes that give the cleanest update of a design block to a target board design.
Parts:
- renumbered C501 to C301, C502 to C302, C503 to C303, L501 to L301, R501 to R301, R502 to R302, U501 to U301
Changed lines of the file:
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@@
 		(in_pos_files yes)
 		(dnp no)
-		(property "Reference" "L501"
+		(property "Reference" "L301"
 			(at 83.82 62.2299 0)
 			(show_name no)
@@
 			)
 			(project "core_board"
-				(path "/efde0c74-5be6-4589-ad87-b4823ac1634b/c87fd2a4-f8d6-4149-89ef-17a7a7e4f014/5463678b-d990-457f-8677-3ee315d0002e"
-					(reference "L501")
+				(path "/efde0c74-5be6-4589-ad87-b4823ac1634b/c87fd2a4-f8d6-4149-89ef-17a7a7e4f014/dad862ba-b1c7-4106-8ed5-6c592a68170e"
+					(reference "L301")
 					(unit 1)
 				)
@@
 		(in_pos_files yes)
 		(dnp no)
-		(property "Reference" "U501"
+		(property "Reference" "U301"
 			(at 96.52 40.64 0)
 			(show_name no)
@@
 			)
 			(project "core_board"
-				(path "/efde0c74-5be6-4589-ad87-b4823ac1634b/c87fd2a4-f8d6-4149-89ef-17a7a7e4f014/5463678b-d990-457f-8677-3ee315d0002e"
-					(reference "U501")
+				(path "/efde0c74-5be6-4589-ad87-b4823ac1634b/c87fd2a4-f8d6-4149-89ef-17a7a7e4f014/dad862ba-b1c7-4106-8ed5-6c592a68170e"
+					(reference "U301")
 					(unit 1)
 				)
@@
 		(in_pos_files yes)
 		(dnp no)
-		(property "Reference" "R501"
+		(property "Reference" "R301"
 			(at 110.49 53.34 90)
 			(show_name no)
@@
 			)
 			(project "core_board"
-				(path "/efde0c74-5be6-4589-ad87-b4823ac1634b/c87fd2a4-f8d6-4149-89ef-17a7a7e4f014/5463678b-d990-457f-8677-3ee315d0002e"
-					(reference "R501")
+				(path "/efde0c74-5be6-4589-ad87-b4823ac1634b/c87fd2a4-f8d6-4149-89ef-17a7a7e4f014/dad862ba-b1c7-4106-8ed5-6c592a68170e"
+					(reference "R301")
 					(unit 1)
 				)
@@
 		(in_pos_files yes)
 		(dnp no)
-		(property "Reference" "R502"
+		(property "Reference" "R302"
 			(at 147.955 51.4349 90)
 			(show_name no)
@@
 			)
 			(project "core_board"
-				(path "/efde0c74-5be6-4589-ad87-b4823ac1634b/c87fd2a4-f8d6-4149-89ef-17a7a7e4f014/5463678b-d990-457f-8677-3ee315d0002e"
-					(reference "R502")
+				(path "/efde0c74-5be6-4589-ad87-b4823ac1634b/c87fd2a4-f8d6-4149-89ef-17a7a7e4f014/dad862ba-b1c7-4106-8ed5-6c592a68170e"
+					(reference "R302")
 					(unit 1)
 				)
@@
 		(in_pos_files yes)
 		(dnp no)
-		(property "Reference" "#PWR0501"
+		(property "Reference" "#PWR0301"
 			(at 96.52 91.44 0)
 			(hide yes)
@@
 			)
 			(project "core_board"
-				(path "/efde0c74-5be6-4589-ad87-b4823ac1634b/c87fd2a4-f8d6-4149-89ef-17a7a7e4f014/5463678b-d990-457f-8677-3ee315d0002e"
-					(reference "#PWR0501")
+				(path "/efde0c74-5be6-4589-ad87-b4823ac1634b/c87fd2a4-f8d6-4149-89ef-17a7a7e4f014/dad862ba-b1c7-4106-8ed5-6c592a68170e"
+					(reference "#PWR0301")
 					(unit 1)
 				)
@@
 		(dnp no)
 		(fields_autoplaced yes)
-		(property "Reference" "#FLG0501"
+		(property "Reference" "#FLG0301"
 			(at 228.6 46.355 0)
 			(hide yes)
@@
 			)
 			(project "core_board"
-				(path "/efde0c74-5be6-4589-ad87-b4823ac1634b/c87fd2a4-f8d6-4149-89ef-17a7a7e4f014/5463678b-d990-457f-8677-3ee315d0002e"
-					(reference "#FLG0501")
+				(path "/efde0c74-5be6-4589-ad87-b4823ac1634b/c87fd2a4-f8d6-4149-89ef-17a7a7e4f014/dad862ba-b1c7-4106-8ed5-6c592a68170e"
+					(reference "#FLG0301")
 					(unit 1)
 				)
@@
 		(in_pos_files yes)
 		(dnp no)
-		(property "Reference" "C501"
+		(property "Reference" "C301"
 			(at 62.23 54.61 0)
 			(show_name no)
@@
 			)
 			(project "core_board"
-				(path "/efde0c74-5be6-4589-ad87-b4823ac1634b/c87fd2a4-f8d6-4149-89ef-17a7a7e4f014/5463678b-d990-457f-8677-3ee315d0002e"
-					(reference "C501")
+				(path "/efde0c74-5be6-4589-ad87-b4823ac1634b/c87fd2a4-f8d6-4149-89ef-17a7a7e4f014/dad862ba-b1c7-4106-8ed5-6c592a68170e"
+					(reference "C301")
 					(unit 1)
 				)
@@
 		(in_pos_files yes)
 		(dnp no)
-		(property "Reference" "C502"
+		(property "Reference" "C302"
 			(at 72.39 54.61 0)
 			(show_name no)
@@
 			)
 			(project "core_board"
-				(path "/efde0c74-5be6-4589-ad87-b4823ac1634b/c87fd2a4-f8d6-4149-89ef-17a7a7e4f014/5463678b-d990-457f-8677-3ee315d0002e"
-					(reference "C502")
+				(path "/efde0c74-5be6-4589-ad87-b4823ac1634b/c87fd2a4-f8d6-4149-89ef-17a7a7e4f014/dad862ba-b1c7-4106-8ed5-6c592a68170e"
+					(reference "C302")
 					(unit 1)
 				)
@@
 		(in_pos_files yes)
 		(dnp no)
-		(property "Reference" "#PWR0502"
+		(property "Reference" "#PWR0302"
 			(at 114.3 76.2 0)
 			(hide yes)
@@
 			)
 			(project "core_board"
-				(path "/efde0c74-5be6-4589-ad87-b4823ac1634b/c87fd2a4-f8d6-4149-89ef-17a7a7e4f014/5463678b-d990-457f-8677-3ee315d0002e"
-					(reference "#PWR0502")
+				(path "/efde0c74-5be6-4589-ad87-b4823ac1634b/c87fd2a4-f8d6-4149-89ef-17a7a7e4f014/dad862ba-b1c7-4106-8ed5-6c592a68170e"
+					(reference "#PWR0302")
 					(unit 1)
 				)
@@
 		(dnp no)
 		(fields_autoplaced yes)
-		(property "Reference" "C503"
+		(property "Reference" "C303"
 			(at 128.27 54.61 0)
 			(show_name no)
@@
 			)
 			(project "core_board"
-				(path "/efde0c74-5be6-4589-ad87-b4823ac1634b/c87fd2a4-f8d6-4149-89ef-17a7a7e4f014/5463678b-d990-457f-8677-3ee315d0002e"
-					(reference "C503")
-					(unit 1)
-				)
+				(path "/efde0c74-5be6-4589-ad87-b4823ac1634b/c87fd2a4-f8d6-4149-89ef-17a7a7e4f014/dad862ba-b1c7-4106-8ed5-6c592a68170e"
+					(reference "C303")
+					(unit 1)
+				)

Commit message: Get core board schematic and layout to pass ERC and DRC. Rework layout to improve organization of components while allowing for future reuse of design.
Parts:
- renumbered C301 to C601, C302 to C602, C303 to C603, L301 to L601, R301 to R601, R302 to R602, U301 to U601
Changed lines of the file:
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@@
 	(wire
 		(pts
-			(xy 140.97 45.72) (xy 140.97 48.26)
+			(xy 140.97 63.5) (xy 140.97 48.26)
 		)
 		(stroke
@@
 	(wire
 		(pts
-			(xy 138.43 45.72) (xy 140.97 45.72)
+			(xy 231.14 63.5) (xy 140.97 63.5)
 		)
 		(stroke
@@
 	(hierarchical_label "BOARD_LOAD_+"
 		(shape output)
-		(at 138.43 45.72 180)
+		(at 231.14 63.5 0)
 		(effects
 			(font
 				(size 1.27 1.27)
 			)
-			(justify right)
+			(justify left)
 		)
 	)
@@
 		(in_pos_files yes)
 		(dnp no)
-		(property "Reference" "L301"
+		(property "Reference" "L601"
 			(at 83.82 62.2299 0)
 			(show_name no)
@@
 			)
 			(project "core_board"
-				(path "/efde0c74-5be6-4589-ad87-b4823ac1634b/c87fd2a4-f8d6-4149-89ef-17a7a7e4f014/67fd60e2-b54e-4371-8a56-a180a344756b"
-					(reference "L301")
+				(path "/efde0c74-5be6-4589-ad87-b4823ac1634b/c87fd2a4-f8d6-4149-89ef-17a7a7e4f014/175829f7-241a-40f0-b17e-c454839fe386"
+					(reference "L601")
 					(unit 1)
 				)
@@
 		(in_pos_files yes)
 		(dnp no)
-		(property "Reference" "U301"
+		(property "Reference" "U601"
 			(at 96.52 40.64 0)
 			(show_name no)
@@
 			)
 			(project "core_board"
-				(path "/efde0c74-5be6-4589-ad87-b4823ac1634b/c87fd2a4-f8d6-4149-89ef-17a7a7e4f014/67fd60e2-b54e-4371-8a56-a180a344756b"
-					(reference "U301")
+				(path "/efde0c74-5be6-4589-ad87-b4823ac1634b/c87fd2a4-f8d6-4149-89ef-17a7a7e4f014/175829f7-241a-40f0-b17e-c454839fe386"
+					(reference "U601")
 					(unit 1)
 				)
@@
 		(in_pos_files yes)
 		(dnp no)
-		(property "Reference" "R301"
+		(property "Reference" "R601"
 			(at 110.49 53.34 90)
 			(show_name no)
@@
 			)
 			(project "core_board"
-				(path "/efde0c74-5be6-4589-ad87-b4823ac1634b/c87fd2a4-f8d6-4149-89ef-17a7a7e4f014/67fd60e2-b54e-4371-8a56-a180a344756b"
-					(reference "R301")
+				(path "/efde0c74-5be6-4589-ad87-b4823ac1634b/c87fd2a4-f8d6-4149-89ef-17a7a7e4f014/175829f7-241a-40f0-b17e-c454839fe386"
+					(reference "R601")
 					(unit 1)
 				)
@@
 		(in_pos_files yes)
 		(dnp no)
-		(property "Reference" "R302"
+		(property "Reference" "R602"
 			(at 147.955 51.4349 90)
 			(show_name no)
@@
 			)
 			(project "core_board"
-				(path "/efde0c74-5be6-4589-ad87-b4823ac1634b/c87fd2a4-f8d6-4149-89ef-17a7a7e4f014/67fd60e2-b54e-4371-8a56-a180a344756b"
-					(reference "R302")
+				(path "/efde0c74-5be6-4589-ad87-b4823ac1634b/c87fd2a4-f8d6-4149-89ef-17a7a7e4f014/175829f7-241a-40f0-b17e-c454839fe386"
+					(reference "R602")
 					(unit 1)
 				)
@@
 		(in_pos_files yes)
 		(dnp no)
-		(property "Reference" "#PWR0301"
+		(property "Reference" "#PWR0601"
 			(at 96.52 91.44 0)
 			(hide yes)
@@
 			)
 			(project "core_board"
-				(path "/efde0c74-5be6-4589-ad87-b4823ac1634b/c87fd2a4-f8d6-4149-89ef-17a7a7e4f014/67fd60e2-b54e-4371-8a56-a180a344756b"
-					(reference "#PWR0301")
+				(path "/efde0c74-5be6-4589-ad87-b4823ac1634b/c87fd2a4-f8d6-4149-89ef-17a7a7e4f014/175829f7-241a-40f0-b17e-c454839fe386"
+					(reference "#PWR0601")
 					(unit 1)
 				)
@@
 		(dnp no)
 		(fields_autoplaced yes)
-		(property "Reference" "#FLG0301"
+		(property "Reference" "#FLG0601"
 			(at 228.6 46.355 0)
 			(hide yes)
@@
 			)
 			(project "core_board"
-				(path "/efde0c74-5be6-4589-ad87-b4823ac1634b/c87fd2a4-f8d6-4149-89ef-17a7a7e4f014/67fd60e2-b54e-4371-8a56-a180a344756b"
-					(reference "#FLG0301")
+				(path "/efde0c74-5be6-4589-ad87-b4823ac1634b/c87fd2a4-f8d6-4149-89ef-17a7a7e4f014/175829f7-241a-40f0-b17e-c454839fe386"
+					(reference "#FLG0601")
 					(unit 1)
 				)
@@
 		(in_pos_files yes)
 		(dnp no)
-		(property "Reference" "C301"
+		(property "Reference" "C601"
 			(at 62.23 54.61 0)
 			(show_name no)
@@
 			)
 			(project "core_board"
-				(path "/efde0c74-5be6-4589-ad87-b4823ac1634b/c87fd2a4-f8d6-4149-89ef-17a7a7e4f014/67fd60e2-b54e-4371-8a56-a180a344756b"
-					(reference "C301")
+				(path "/efde0c74-5be6-4589-ad87-b4823ac1634b/c87fd2a4-f8d6-4149-89ef-17a7a7e4f014/175829f7-241a-40f0-b17e-c454839fe386"
+					(reference "C601")
 					(unit 1)
 				)
@@
 		(in_pos_files yes)
 		(dnp no)
-		(property "Reference" "C302"
+		(property "Reference" "C602"
 			(at 72.39 54.61 0)
 			(show_name no)
@@
 			)
 			(project "core_board"
-				(path "/efde0c74-5be6-4589-ad87-b4823ac1634b/c87fd2a4-f8d6-4149-89ef-17a7a7e4f014/67fd60e2-b54e-4371-8a56-a180a344756b"
-					(reference "C302")
+				(path "/efde0c74-5be6-4589-ad87-b4823ac1634b/c87fd2a4-f8d6-4149-89ef-17a7a7e4f014/175829f7-241a-40f0-b17e-c454839fe386"
+					(reference "C602")
 					(unit 1)
 				)
@@
 		(in_pos_files yes)
 		(dnp no)
-		(property "Reference" "#PWR0302"
+		(property "Reference" "#PWR0602"
 			(at 114.3 76.2 0)
 			(hide yes)
@@
 			)
 			(project "core_board"
-				(path "/efde0c74-5be6-4589-ad87-b4823ac1634b/c87fd2a4-f8d6-4149-89ef-17a7a7e4f014/67fd60e2-b54e-4371-8a56-a180a344756b"
-					(reference "#PWR0302")
+				(path "/efde0c74-5be6-4589-ad87-b4823ac1634b/c87fd2a4-f8d6-4149-89ef-17a7a7e4f014/175829f7-241a-40f0-b17e-c454839fe386"
+					(reference "#PWR0602")
 					(unit 1)
 				)
@@
 		(dnp no)
 		(fields_autoplaced yes)
-		(property "Reference" "C303"
+		(property "Reference" "C603"
 			(at 128.27 54.61 0)
 			(show_name no)
@@
 			)
 			(project "core_board"
-				(path "/efde0c74-5be6-4589-ad87-b4823ac1634b/c87fd2a4-f8d6-4149-89ef-17a7a7e4f014/67fd60e2-b54e-4371-8a56-a180a344756b"
-					(reference "C303")
-					(unit 1)
-				)
+				(path "/efde0c74-5be6-4589-ad87-b4823ac1634b/c87fd2a4-f8d6-4149-89ef-17a7a7e4f014/175829f7-241a-40f0-b17e-c454839fe386"
+					(reference "C603")
+					(unit 1)
+				)
